File: hardware/PCB/Sensors1.kicad_sch (KiCad schematic)
At the start: 29 parts, among them J10 WCS1800, J101 INA333, J11 INA333, J12 Micro SD Adapter, J13 Relays, J201 Micro_SD_Card_Det2, J202 Screw_Terminal_01x03, K201 SANYOU_SRD_Form_C, Q201 NPN, U101 INA333xxDGK, U201 QNHC3, U202 PC817C

Commit message: test com
Other:
- note added: "test"
Changed lines of the file:
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@@
+		)
+	)
+	(text "test"
+		(exclude_from_sim no)
+		(at 139.7 82.042 0)
+		(effects
+			(font
+				(size 1.27 1.27)
+			)
 		)
 	)

Commit message: pcb commit
Parts:
- added D2, D4: 1N4148, Diode_SMD:D_SOD-323, symbol Device:D
- added J14, J6: Screw_Terminal_01x03, symbol Connector:Screw_Terminal_01x03
- added K1, K2: SANYOU_SRD_Form_C, Relay_THT:Relay_SPDT_SANYOU_SRD_Series_Form_C, symbol Relay:SANYOU_SRD_Form_C
- added Q1, Q3: NPN, symbol Simulation_SPICE:NPN
- added R1, R2, R7, R8: 220R, Resistor_SMD:R_0805_2012Metric, symbol Device:R
- added U2, U5: PC817C, symbol Isolator:VO615A
- D201: value D -> 1N4148; footprint (none) -> Diode_SMD:D_SOD-323; LCSC (none) -> C2128
Connections:
- net !!!!: now also R2.1, R8.1, U2.3, U5.3
- net +3V3: now also D2.1 (K), D4.1 (K), K1.5, K2.5, U2.4, U5.4
- net GND: now also Q1.3 (E), Q3.3 (E), U2.2, U5.2
- net R1IN1 renamed R1_IN1
- net R1IN2 renamed R1_IN2
- net R1_IN2: now also R1.1
- net R1IN3 renamed R1_IN3
- net R1_IN3: now also R7.1
- new net: Q1.2 (B), R2.2
- new net: D2.2 (A), K2.2, Q3.1 (C)
- new net: R1.2, U2.1
- new net: J14.1 (Pin_1), K2.4
- new net: J14.2 (Pin_2), K2.1
- new net: J14.3 (Pin_3), K2.3
- new net: R7.2, U5.1
- new net: J6.2 (Pin_2), K1.1
- new net: D4.2 (A), K1.2, Q1.1 (C)
- new net: J6.3 (Pin_3), K1.3
- new net: J6.1 (Pin_1), K1.4
- new net: Q3.2 (B), R8.2
Other:
- note added: "Przerwane w trakcie roboty dodać footprinty"
- note removed: "https://piotr-gorecki.pl/yk012-wspolnie-projektujemy-uniwersalne-obciazenie-aktywne/"
- note removed: "lm358 irlz44n 10uF R = 1kohm ? Rs = 1ohm"
- note removed: "test"
- moved on the sheet: D201, J13, J202, K201, Q201, R201, R202, U202

Commit message: PCB
Parts:
- removed C208: 100n, Capacitor_SMD:C_0805_2012Metric, symbol Device:C
- removed D2, D201, D4: 1N4148, Diode_SMD:D_SOD-323, symbol Device:D
- removed J12: Micro SD Adapter, Connector_PinHeader_2.54mm:PinHeader_1x06_P2.54mm_Vertical, symbol Connector:Conn_01x06_Pin
- removed J13: Relays, Connector_PinHeader_2.54mm:PinHeader_1x06_P2.54mm_Vertical, symbol Connector:Conn_01x06_Pin
- removed J14, J202, J6: Screw_Terminal_01x03, symbol Connector:Screw_Terminal_01x03
- removed J201: Micro_SD_Card_Det2, symbol Connector:Micro_SD_Card_Det2
- removed JP202: SolderJumper_2_Open, Jumper:SolderJumper-2_P1.3mm_Open_TrianglePad1.0x1.5mm, symbol Jumper:SolderJumper_2_Open
- removed K1, K2, K201: SANYOU_SRD_Form_C, Relay_THT:Relay_SPDT_SANYOU_SRD_Series_Form_C, symbol Relay:SANYOU_SRD_Form_C
- removed Q1, Q201, Q3: NPN, symbol Simulation_SPICE:NPN
- removed R1, R2, R201, R202, R7, R8: 220R, Resistor_SMD:R_0805_2012Metric, symbol Device:R
- removed R101: 100R, Resistor_SMD:R_0805_2012Metric, symbol Device:R
- removed R102, R103: 10k, Resistor_SMD:R_0805_2012Metric, symbol Device:R
- removed U2, U202, U5: PC817C, symbol Isolator:VO615A
- added C2: 10u, Capacitor_SMD:C_1206_3216Metric, symbol Device:C
- added C202: 100n, Capacitor_SMD:C_0805_2012Metric, symbol Device:C
- added J_BAT1: Conn_01x02, TerminalBlock:TerminalBlock_MaiXu_MX126-5.0-02P_1x02_P5.00mm, symbol Connector_Generic:Conn_01x02
- added Q2: IRLZ44N, Package_TO_SOT_THT:TO-220-3_Vertical, symbol Transistor_FET:IRLZ44N
- added R5: 1k, Resistor_SMD:R_0805_2012Metric, symbol Device:R
- added R6: 1R, symbol Device:R
- added U103, U4: LM358, footprints:LM358, symbol Amplifier_Operational:LM358
- C101, C102, C103: Manufacturer (none) -> Samsung Electro-Mechanics
- C201: Distributor https://jlcpcb.com/partdetail/28983-CL21B104KCFNNNE/C28233 -> (none); JLCPCB Part (none) -> C28233; Link (none) -> https://jlcpcb.com/partdetail/28983-CL21B104KCFNNNE/C28233
- D202, D203: Distributor https://jlcpcb.com/partdetail/DiodesIncorporated-MMSZ5226BS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 -> (none); Link (none) -> https://jlcpcb.com/partdetail/DiodesIncorporated-MMSZ5226BS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
- J10, J101, J11: JLCPCB Part (none) -> C2337; LCSC C2337 -> (none)
- R203, R204: Distributor https://jlcpcb.com/partdetail/28584-0805W8F5101T5E/C27834 -> (none); Link (none) -> https://jlcpcb.com/partdetail/28584-0805W8F5101T5E/C27834
- renumbered U101 to U102
Connections:
- net +3V3: no longer C101.1, J10.1 (Pin_1), U102.7 (V+), U201.3 (Vcc)
- net GND: now also C2.2, C202.2, J_BAT1.2 (Pin_2), R6.1, U4.4 (V-)
- net QNH_out: now also C202.1
- new net: C2.1, R5.2, U4.3 (+)
- new net: Q2.1 (G), U4.1
- new net: Q2.3 (S), R6.2, U4.2 (-)
- new net +5V: C101.1, U102.7 (V+), U201.3 (Vcc), U4.8 (V+)
- new net VCC: J10.1 (Pin_1)
- new net battery_load: J_BAT1.1 (Pin_1), Q2.2 (D)
- new net pwm_current_sel: R5.1
- no-connect marks 4 -> 8
Other:
- note added: "Bat+"
- note added: "Bat-"
- note added: "I=U_{PWM}/R"
- note added: "https://piotr-gorecki.pl/yk012-wspolnie-projektujemy-uniwersalne-obciazenie-aktywne/"
- note removed: "CS_SD karta"
- note removed: "Przerwane w trakcie roboty dodać footprinty"
- note removed: "i THT na moduł i na smd"
- note removed: "jaks popularna obudowa karty micor sd połączneia z kartą na płytce i wyjscia na zewnętrzny moduł solder brige tylk na CS na plytce"
- moved on the sheet: C101, C102, C103, D202, J10, J101, J11, JP201, R204, U102, U201

Commit message: PCB
Parts:
- removed C101, C102, C103: 0.1u, Capacitor_SMD:C_0805_2012Metric, symbol Device:C
- removed C2: 10u, Capacitor_SMD:C_1206_3216Metric, symbol Device:C
- removed C201, C202: 100n, Capacitor_SMD:C_0805_2012Metric, symbol Device:C
- removed D202, D203: 3.3V, Diode_SMD:D_SOD-323, symbol Device:D_Schottky
- removed J10: WCS1800, Connector_PinHeader_2.54mm:PinHeader_1x04_P2.54mm_Vertical, symbol Connector:Conn_01x04_Pin
- removed J_BAT1: Conn_01x02, TerminalBlock:TerminalBlock_MaiXu_MX126-5.0-02P_1x02_P5.00mm, symbol Connector_Generic:Conn_01x02
- removed Q2: IRLZ44N, Package_TO_SOT_THT:TO-220-3_Vertical, symbol Transistor_FET:IRLZ44N
- removed R203, R204: 5.1k, Resistor_SMD:R_0805_2012Metric, symbol Device:R
- removed R5: 1k, Resistor_SMD:R_0805_2012Metric, symbol Device:R
- removed U103, U4: LM358, footprints:LM358, symbol Amplifier_Operational:LM358
- added C1, C10, C11, C3, C5, C6, C7: 100n, Capacitor_SMD:C_0805_2012Metric, symbol Device:C
- added C4: 1n, Capacitor_SMD:C_0805_2012Metric, symbol Device:C
- added C8, C9: 1u, Capacitor_SMD:C_0805_2012Metric, symbol Device:C
- added J10: Conn_ACS712, symbol Connector:Conn_01x03_Socket
- added JP1: SolderJumper_3_Open, Jumper:SolderJumper-3_P2.0mm_Open_TrianglePad1.0x1.5mm_NumberLabels, symbol Jumper:SolderJumper_3_Open
- added R10, R11: 6.2k, Resistor_SMD:R_0805_2012Metric, symbol Device:R
- added R13: 2.2k, Resistor_SMD:R_0805_2012Metric, symbol Device:R
- added R14, R20, R22, R23, R25: 10k, Resistor_SMD:R_0805_2012Metric, symbol Device:R
- added R16, R17: 4.7k, Resistor_SMD:R_0805_2012Metric, symbol Device:R
- added R18, R19: 8.2k, Resistor_SMD:R_0805_2012Metric, symbol Device:R
- added R9: 3.9k, Resistor_SMD:R_0805_2012Metric, symbol Device:R
- added U1: MCP6002T-I/SN, Package_SO:SOIC-8_3.9x4.9mm_P1.27mm, symbol Amplifier_Operational:MCP6002-xSN
- added U6: ACS712xLCTR-05B, Package_SO:SOIC-8_3.9x4.9mm_P1.27mm, symbol Sensor_Current:ACS712xLCTR-05B
- added U7, U8: TLV431, Package_TO_SOT_SMD:SOT-23, symbol Reference_Voltage:REF3012
- added U9: BME280, Package_LGA:Bosch_LGA-8_2.5x2.5mm_P0.65mm_ClockwisePinNumbering, symbol Sensor:BME280
- R6: value 1R -> 3.9k; footprint (none) -> Resistor_SMD:R_0805_2012Metric; JLCPCB Part (none) -> C17614; Link (none) -> https://jlcpcb.com/partdetail/18302-0805W8F3901T5E/C17614; MFR Part (none) -> 0805W8F3901T5E; Manufacturer (none) -> UNI-ROYAL(Uniroyal Elec); now in the parts list
Connections:
- net +3V3: now also C10.1, C11.1, R22.1, R23.1, U1.8 (V+), U9.6 (VDDIO), U9.8 (VDD)
- net +5V: now also C1.1, C3.1, C7.1, J10.1 (Pin_1), U6.8 (VCC)
- net GND: now also C1.2, C10.2, C11.2, C3.2, C4.2, C5.2, C6.2, C7.2, C8.2, C9.2, J10.3 (Pin_3), R10.2, R18.2, R20.2, R25.2, U1.4 (V-), U6.5 (GND), U7.3 (GND), U8.3 (GND), U9.1 (GND), U9.7 (GND); no longer R6.1
- net QNH_out: now also R19.1, U1.7
- net ina333_Vin+: now also C5.1
- net ina333_Vin-: now also C6.1
- net ina333_Vout: now also R11.1, U1.1
- net ina333_Vout_5V: now also R6.1
- net ina333_opamp_V+: now reaches R6.2
- net ina333_opamp_V+: now also R10.1, R11.2, R9.2, U1.2 (-), U1.3 (+)
- net QNHC3_out: now reaches U201.1 (OUT)
- net QNHC3_out: now also JP1.3 (B)
- new net: R14.2, R25.1, U8.2 (OUT)
- new net: R13.2, R20.1, U7.2 (OUT)
- new net: C4.1, U6.6 (FILTER)
- new net ACS712_out: J10.2 (Pin_2), JP1.1 (A), U6.7 (VIOUT)
- new net BME280_SPI_CLK: U9.4 (SCK)
- new net BME280_SPI_MISO: U9.5 (SDO)
- new net BME282_SPI_MOSI: U9.3 (SDI)
- new net BME283_SPI_CS: U9.2 (CSB)
- new net Current_offset_1V5: C8.1, R13.1, R16.1, R23.2, U7.1 (IN)
- new net Current_opamp_V+: R16.2, R17.2, R18.1, R19.2, U1.5 (+), U1.6 (-)
- new net Current_sensor_in+: U6.1 (IP+), U6.2 (IP+)
- new net Current_sensor_in-: U6.3 (IP-), U6.4 (IP-)
- new net Current_sensor_out: JP1.2 (C), R17.1
- new net ina333_offset_2V48: C9.1, R14.1, R22.2, R9.1, U8.1 (IN)
- no-connect marks 8 -> 2
Other:
- note added: "0.344 mV/A gain = 1.74 offset = 1.5V <-5A; 5A>"
- note added: "185 mV/A -5A = 2.5-(0.185*5) = 1.575V 0A = 2.5V 5A = 2.5+(0.185*5) = 3.425V"
- note added: "Internal Vref = 1.24V Vout = (1 + R1/R2)*Vref = 1.5128V"
- note added: "Internal Vref = 1.24V Vout = (1 + R1/R2)*Vref = 2.48V"
- note added: "QNHC3/ACS712"
- note added: "gain = 1.58 offset = 2.48V <2.48V; 4.55V>"
- note removed: "ACS712"
- note removed: "Bat+"
- note removed: "Bat-"
- note removed: "D"
- note removed: "I=U_{PWM}/R"
- note removed: "QNHC3"
- note removed: "https://piotr-gorecki.pl/yk012-wspolnie-projektujemy-uniwersalne-obciazenie-aktywne/"
- note removed: "ja tu wstawie piny z mojeo sensora co mam"
- moved on the sheet: J101, J11, JP201, U102, U201

Commit message: pcb sensors
Parts:
- added R12: R, symbol Device:R
Other:
- moved on the sheet: C1, U201
Changed lines of the file:
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@@
 	)
 	(junction
-		(at 48.26 81.28)
+		(at 44.45 82.55)
 		(diameter 0)
 		(color 0 0 0 0)
@@
 	(wire
 		(pts
-			(xy 55.88 83.82) (xy 46.99 83.82)
+			(xy 52.07 85.09) (xy 43.18 85.09)
 		)
 		(stroke
@@
 	(wire
 		(pts
-			(xy 48.26 71.12) (xy 57.15 71.12)
+			(xy 44.45 72.39) (xy 53.34 72.39)
 		)
 		(stroke
@@
 	(wire
 		(pts
-			(xy 48.26 71.12) (xy 48.26 81.28)
+			(xy 44.45 72.39) (xy 44.45 82.55)
 		)
 		(stroke
@@
 	(wire
 		(pts
-			(xy 48.26 86.36) (xy 46.99 86.36)
+			(xy 44.45 87.63) (xy 43.18 87.63)
 		)
 		(stroke
@@
 	(wire
 		(pts
-			(xy 48.26 81.28) (xy 46.99 81.28)
+			(xy 44.45 82.55) (xy 43.18 82.55)
 		)
 		(stroke
@@
 	)
 	(label "QNHC3_out"
-		(at 55.88 83.82 0)
+		(at 52.07 85.09 0)
 		(effects
 			(font
@@
 	(symbol
 		(lib_id "Device:C")
-		(at 57.15 74.93 0)
+		(at 53.34 76.2 0)
 		(mirror y)
 		(unit 1)
@@
 		(dnp no)
 		(property "Reference" "C1"
-			(at 54.61 73.66 0)
+			(at 50.8 74.93 0)
 			(effects
 				(font
@@
 		)
 		(property "Value" "100n"
-			(at 54.61 76.2 0)
+			(at 50.8 77.47 0)
 			(effects
 				(font
@@
 		)
 		(property "Footprint" "Capacitor_SMD:C_0805_2012Metric"
-			(at 56.1848 78.74 0)
+			(at 52.3748 80.01 0)
 			(effects
 				(font
@@
 		)
 		(property "Datasheet" "~"
-			(at 57.15 74.93 0)
+			(at 53.34 76.2 0)
 			(effects
 				(font
@@
 		)
 		(property "Description" "Unpolarized capacitor"
-			(at 57.15 74.93 0)
+			(at 53.34 76.2 0)
 			(effects
 				(font
@@
 		)
 		(property "MFR Part" "CL21B104KCFNNNE"
-			(at 57.15 74.93 0)
+			(at 53.34 76.2 0)
 			(effects
 				(font
@@
 		)
 		(property "Manufacturer" "Samsung Electro-Mechanics"
-			(at 57.15 74.93 0)
+			(at 53.34 76.2 0)
 			(effects
 				(font
@@
 		)
 		(property "Link" "https://jlcpcb.com/partdetail/28983-CL21B104KCFNNNE/C28233"
-			(at 57.15 74.93 0)
+			(at 53.34 76.2 0)
 			(effects
 				(font
@@
 		)
 		(property "JLCPCB Part" "C28233"
-			(at 57.15 74.93 0)
+			(at 53.34 76.2 0)
 			(effects
 				(font
@@
 	)
 	(symbol
+		(lib_id "Device:R")
+		(at 64.77 35.56 0)
+		(unit 1)
+		(exclude_from_sim no)
+		(in_bom yes)
+		(on_board yes)
+		(dnp no)
+		(fields_autoplaced yes)
+		(property "Reference" "R12"
+			(at 67.31 34.2899 0)
+			(effects
+				(font
+					(size 1.27 1.27)
+				)
+				(justify left)
+			)
+		)
+		(property "Value" "R"
+			(at 67.31 36.8299 0)
+			(effects
+				(font
+					(size 1.27 1.27)
+				)
+				(justify left)
+			)
+		)
+		(property "Footprint" ""
+			(at 62.992 35.56 90)
+			(effects
+				(font
+					(size 1.27 1.27)
+				)
+				(hide yes)
+			)
+		)
+		(property "Datasheet" "~"
+			(at 64.77 35.56 0)
+			(effects
+				(font
+					(size 1.27 1.27)
+				)
+				(hide yes)
+			)
+		)
+		(property "Description" "Resistor"
+			(at 64.77 35.56 0)
+			(effects
+				(font
+					(size 1.27 1.27)
+				)
+				(hide yes)
+			)
+		)
+		(pin "1"
+		)
+		(pin "2"
+		)
+		(instances
+			(project ""
+				(path "/3ad3be82-7cab-4f72-ad1b-fa82ddc3a5e0/0d146a7f-c55b-4837-864c-e0f7f24def8d"
+					(reference "R12")
+					(unit 1)
+				)
+			)
+		)
+	)
+	(symbol
 		(lib_id "power:GND")
 		(at 237.49 120.65 0)
@@
 	(symbol
 		(lib_id "power:GND")
-		(at 57.15 78.74 0)
+		(at 53.34 80.01 0)
 		(mirror y)
 		(unit 1)
@@
 		(fields_autoplaced yes)
 		(property "Reference" "#PWR036"
-			(at 57.15 85.09 0)
+			(at 53.34 86.36 0)
 			(effects
 				(font
@@
 		)
 		(property "Value" "GND"
-			(at 57.15 83.82 0)
+			(at 53.34 85.09 0)
 			(effects
 				(font
@@
 		)
 		(property "Footprint" ""
-			(at 57.15 78.74 0)
+			(at 53.34 80.01 0)
 			(effects
 				(font
@@
 		)
 		(property "Datasheet" ""
-			(at 57.15 78.74 0)
+			(at 53.34 80.01 0)
 			(effects
 				(font
@@
 		)
 		(property "Description" "Power symbol creates a global label with name \"GND\" , ground"
-			(at 57.15 78.74 0)
+			(at 53.34 80.01 0)
 			(effects
 				(font
@@
 	(symbol
 		(lib_id "footprints:QNHC3")
-		(at 41.91 82.55 0)
+		(at 38.1 83.82 0)
 		(mirror y)
 		(unit 1)
@@
 		(dnp no)
 		(property "Reference" "U201"
-			(at 38.1 82.4229 0)
+			(at 34.29 83.6929 0)
 			(effects
 				(font
@@
 		)
 		(property "Value" "QNHC3"
-			(at 38.1 84.9629 0)
+			(at 34.29 86.2329 0)
 			(effects
 				(font
@@
 		)
 		(property "Footprint" "footprints:QNHC3"
-			(at 41.91 82.55 0)
+			(at 38.1 83.82 0)
 			(effects
 				(font
@@
 		)
 		(property "Datasheet" "https://pl.aliexpress.com/item/1005006113864778.html?gatewayAdapt=glo2pol"
-			(at 41.91 82.55 0)
+			(at 38.1 83.82 0)
 			(effects
 				(font
@@
 		)
 		(property "Description" ""
-			(at 41.91 82.55 0)
+			(at 38.1 83.82 0)
 			(effects
 				(font
@@
 	(symbol
 		(lib_id "power:+5V")
-		(at 48.26 81.28 270)
+		(at 44.45 82.55 270)
 		(mirror x)
 		(unit 1)
@@
 		(dnp no)
 		(property "Reference" "#PWR0201"
-			(at 44.45 81.28 0)
+			(at 40.64 82.55 0)
 			(effects
 				(font
@@
 		)
 		(property "Value" "+5V"
-			(at 52.832 81.28 90)
+			(at 49.022 82.55 90)
 			(effects
 				(font
@@
 		)
 		(property "Footprint" ""
-			(at 48.26 81.28 0)
+			(at 44.45 82.55 0)
 			(effects
 				(font
@@
 		)
 		(property "Datasheet" ""
-			(at 48.26 81.28 0)
+			(at 44.45 82.55 0)
 			(effects
 				(font
@@
 		)
 		(property "Description" "Power symbol creates a global label with name \"+5V\""
-			(at 48.26 81.28 0)
+			(at 44.45 82.55 0)
 			(effects
 				(font
@@
 	(symbol
 		(lib_id "power:GND")
-		(at 48.26 86.36 90)
+		(at 44.45 87.63 90)
 		(mirror x)
 		(unit 1)
@@
 		(fields_autoplaced yes)
 		(property "Reference" "#PWR0202"
-			(at 54.61 86.36 0)
+			(at 50.8 87.63 0)
 			(effects
 				(font
@@
 		)
 		(property "Value" "GND"
-			(at 53.34 86.36 0)
+			(at 49.53 87.63 0)
 			(effects
 				(font
@@
 		)
 		(property "Footprint" ""
-			(at 48.26 86.36 0)
+			(at 44.45 87.63 0)
 			(effects
 				(font
@@
 		)
 		(property "Datasheet" ""
-			(at 48.26 86.36 0)
+			(at 44.45 87.63 0)
 			(effects
 				(font
@@
 		)
 		(property "Description" "Power symbol creates a global label with name \"GND\" , ground"
-			(at 48.26 86.36 0)
+			(at 44.45 87.63 0)
 			(effects
 				(font
