File: hardware/PCB/Connectors.kicad_sch (KiCad schematic)
At the start: 5 parts, among them J4 J_OLED, J5 J_SGP30, J7 J_BMP1, J8 J_BMP2, J9 J_BMP3

Commit message: pcb sensors
Parts:
- removed J9: J_BMP3, Connector_PinHeader_2.54mm:PinHeader_1x06_P2.54mm_Vertical, symbol Connector:Conn_01x06_Pin
- added C104, C105, C106, C107, C109, C110: 100n, Capacitor_SMD:C_0805_2012Metric, symbol Device:C
- added C108: 2.2u, Capacitor_SMD:C_0805_2012Metric, symbol Device:C
- added D101: D_Schottky_3A, Diode_SMD:D_SMA, symbol Device:D_Schottky
- added F201: xA, Fuse:Fuseholder_Clip-5x20mm_Littelfuse_111_Inline_P20.00x5.00mm_D1.05mm_Horizontal, symbol Device:Polyfuse
- added FID1, FID2, FID3, FID4: Fiducial, Fiducial:Fiducial_1mm_Mask2mm, symbol Mechanical:Fiducial
- added H1, H2, H3, H4: MountingHole_Pad, MountingHole:MountingHole_3.2mm_M3_Pad, symbol Mechanical:MountingHole_Pad
- added J103: enc, Connector_PinHeader_2.54mm:PinHeader_1x05_P2.54mm_Vertical, symbol Connector:Conn_01x05_Pin
- added J104: Barrel_Jack_Switch_Pin3Ring, Connector_BarrelJack:BarrelJack_GCT_DCJ200-10-A_Horizontal, symbol Connector:Barrel_Jack_Switch_Pin3Ring
- added J3: USB_C_Receptacle_USB2.0_16P, Connector_USB:USB_C_Receptacle_GCT_USB4105-xx-A_16P_TopMnt_Horizontal, symbol Connector:USB_C_Receptacle_USB2.0_16P
- added L101: 2.2uH, Inductor_SMD:L_Sunlord_MWSA0503S, symbol Device:L
- added R104, R105, R106, R3, R4: 5.1k, Resistor_SMD:R_0805_2012Metric, symbol Device:R
- added R107: 100k, Resistor_SMD:R_0805_2012Metric, symbol Device:R
- added R108: 22.1k, Resistor_SMD:R_0805_2012Metric, symbol Device:R
- added U101: LMR51430, Package_TO_SOT_SMD:SOT-23-6, symbol Regulator_Switching:LMR51430
- added U104: ~, footprints:board_step-down, symbol footprints:board_step-down
- added U3: USBLC6-2SC6, Package_TO_SOT_SMD:SOT-23-6, symbol Power_Protection:USBLC6-2SC6
Connections:
- net +3V3: now also C110.2, J103.1 (Pin_1), L101.2, R107.1, U104.2 (OUT+); no longer J4.8 (Pin_8)
- net GND: now also C104.2, C105.2, C106.2, C108.2, C109.2, C110.1, H1.1, H2.1, H3.1, H4.1, J103.5 (Pin_5), J104.2, J104.3, J3.A1 (GND), J3.A12 (GND), J3.B1 (GND), J3.B12 (GND), J3.S1 (SHIELD), R108.2, R3.2, R4.2, U101.1 (GND), U104.3 (IN-), U104.4 (OUT-), U3.2 (GND)
- net BMP1_CS_B5 renamed BMP1_CS
- net I2C_SCL_B6 renamed I2C_SCL
- net I2C_SDA_B9 renamed I2C_SDA
- net OLED_CS_A1 renamed OLED_CS
- net OLED_DC_A2 renamed OLED_DC
- net OLED_RST_A3 renamed OLED_RST
- net SPI_MISO_A6 renamed SPI_MISO
- net SPI_MOSI_A7 renamed SPI_MOSI
- net SPI_SCK_A5 renamed SPI_SCK
- new net: J3.A4 (VBUS), J3.A9 (VBUS), J3.B4 (VBUS), J3.B9 (VBUS), U3.5 (VBUS)
- new net: D101.1 (K), F201.1
- new net: D101.2 (A), J104.1
- new net +5V: C108.1, C109.1, F201.2, U101.3 (VIN), U101.5 (EN), U104.1 (IN+)
- new net SMPS_CB: C107.2, U101.6 (CB)
- new net SMPS_FB: R107.2, R108.1, U101.4 (FB)
- new net SMPS_SW: C107.1, L101.1, U101.2 (SW)
- new net USBCC1: J3.A5 (CC1), R4.1
- new net USBCC2: J3.B5 (CC2), R3.1
- new net USBD+: J3.A6 (D+), J3.B6 (D+), U3.3 (I/O2)
- new net USBD-: J3.A7 (D-), J3.B7 (D-), U3.1 (I/O1)
- new net USB_D+: U3.4 (I/O2)
- new net USB_D-: U3.6 (I/O1)
- new net enc_KEY: C106.1, R106.2
- new net enc_S1: C104.1, R104.2
- new net enc_S1_in: J103.4 (Pin_4), R104.1
- new net enc_S2: C105.1, R105.2
- new net enc_S2_in: J103.3 (Pin_3), R105.1
- new net enc_key_in: J103.2 (Pin_2), R106.1
- no-connect marks 5 -> 7
Other:
- note added: "5.0V -> 3.3V"
- note added: "USB-C"
- note added: "encoder"
- note removed: "dupont 2.54mm"
- moved on the sheet: J4, J5, J7, J8

Commit message: Rough Layout pcb
Parts:
- removed J4: J_OLED, Connector_PinHeader_2.54mm:PinHeader_1x14_P2.54mm_Vertical, symbol Connector:Conn_01x14_Pin
- added C408: 100n, Capacitor_SMD:C_0805_2012Metric, symbol Device:C
- added C409: 1u, Capacitor_SMD:C_0805_2012Metric, symbol Device:C
- added J408: J_OLED, Connector_JST:JST_XH_B9B-XH-A_1x09_P2.50mm_Vertical, symbol Connector:Conn_01x09_Pin
- added J409: Conn_01x05_Pin, Connector_JST:JST_XH_B5B-XH-A_1x05_P2.50mm_Vertical, symbol Connector:Conn_01x05_Pin
- added J410: Micro SD, footprints:board_smd_sd, symbol Connector:Conn_01x08_Pin
- added J411: Micro SD2, Connector_PinHeader_2.54mm:PinHeader_1x08_P2.54mm_Vertical, symbol Connector:Conn_01x08_Socket
- added J412: Micro_SD_Card, footprints:microSD, symbol Connector:Micro_SD_Card
- added R408, R409, R410, R411, R412: 10k, Resistor_SMD:R_0805_2012Metric, symbol Device:R
- added TP401, TP402, TP403: TestPoint, TestPoint:TestPoint_Pad_D1.5mm, symbol Connector:TestPoint
- F401: renamed from F201; now in the parts list
- J401: renamed from J5; footprint (none) -> Connector_JST:JST_XH_B4B-XH-A_1x04_P2.50mm_Vertical; Link (none) -> https://pl.aliexpress.com/item/1005010374454394.html?spm=a2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; now left out of the parts list
- J402: renamed from J3; JLCPCB Part (none) -> C3025063; MFR Part (none) -> USB4105-GF-A-060; Manufacturer (none) -> Global Connector Technology
- J403: renamed from J104; value Barrel_Jack_Switch_Pin3Ring -> 5V; Link (none) -> https://pl.aliexpress.com/item/33005175186.html?spm=a2g0o.p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
- J404: renamed from J7; footprint Connector_PinHeader_2.54mm:PinHeader_1x06_P2.54mm_Vertical -> Connector_JST:JST_XH_B6B-XH-A_1x06_P2.50mm_Vertical; JLCPCB Part C2337 -> (none); Link (none) -> https://pl.aliexpress.com/item/1005006960863510.html?spm=a2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; now left out of the parts list
- J405: renamed from U104; Link (none) -> https://pl.aliexpress.com/item/1005010319587802.html?spm=a2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; now left out of the parts list
- J406: renamed from J8; footprint Connector_PinHeader_2.54mm:PinHeader_1x06_P2.54mm_Vertical -> Connector_JST:JST_XH_B6B-XH-A_1x06_P2.50mm_Vertical; JLCPCB Part C2337 -> (none); Link (none) -> https://pl.aliexpress.com/item/1005006960863510.html?spm=a2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; now left out of the parts list
- J407: renamed from J103; footprint Connector_PinHeader_2.54mm:PinHeader_1x05_P2.54mm_Vertical -> Connector_JST:JST_XH_B5B-XH-A_1x05_P2.50mm_Vertical; JLCPCB Part C2337 -> (none); now left out of the parts list
- R401: renamed from R4; JLCPCB Part (none) -> C27834
- R402: renamed from R3; JLCPCB Part (none) -> C27834
- R405: renamed from R106; JLCPCB Part (none) -> C27834
- R406: renamed from R105; JLCPCB Part (none) -> C27834
- R407: renamed from R104; JLCPCB Part (none) -> C27834
- U401: renamed from U3; JLCPCB Part (none) -> C7519; MFR Part (none) -> USBLC6-2SC6; Manufacturer (none) -> STMicroelectronics
- renumbered C107 to C401, C108 to C402, C109 to C403, C110 to C404, C104 to C405, C105 to C406, C106 to C407, D101 to D401, FID1 to FID401, FID2 to FID402, FID3 to FID403, FID4 to FID404, H1 to H401, H2 to H402, H3 to H403, H4 to H404, L101 to L401, R107 to R403, R108 to R404, U101 to U402
Connections:
- net +3V3: now also C404.1, C408.1, C409.1, J408.1 (Pin_1), J410.7 (Pin_7), J411.7 (Pin_7), J412.4 (VDD), R408.1, R409.1, R410.1, R411.1, R412.1, TP402.1; no longer C404.2
- net +5V: now also TP403.1
- net GND: now also C404.2, C408.2, C409.2, J408.2 (Pin_2), J410.6 (Pin_6), J411.6 (Pin_6), J412.6 (VSS); no longer C404.1
- net OLED_CS: now also J408.3 (Pin_3)
- net OLED_DC: now also J408.5 (Pin_5)
- net OLED_RST: now also J408.4 (Pin_4)
- net SPI_MISO: now also J408.9 (Pin_9), J410.2 (Pin_2), J411.2 (Pin_2), J412.7 (DAT0), R411.2
- net SPI_MOSI: now also J408.6 (Pin_6), J410.4 (Pin_4), J411.4 (Pin_4), J412.3 (CMD), R410.2
- net SPI_SCK: now also J408.7 (Pin_7), J410.3 (Pin_3), J411.3 (Pin_3), J412.5 (CLK)
- net at D401.2 (A), J403.1: now also TP401.1
- new net: J412.8 (DAT1), R412.2
- new net: J412.1 (DAT2), R408.2
- new net OLED_TIM2: J408.8 (Pin_8)
- new net SD_CS: J410.5 (Pin_5), J411.5 (Pin_5), J412.2 (DAT3/CD), R409.2
- no-connect marks 7 -> 12
Other:
- note added: "microSD"
- moved on the sheet: C405, C406, C407, FID401, FID402, FID403, FID404, H401, H402, H403, H404, J401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

Commit message: XL4015 CC, relays
Parts:
- D401: value D_Schottky_3A -> D_Schottky_5A
- F401: value xA -> 5A; footprint Fuse:Fuseholder_Clip-5x20mm_Littelfuse_111_Inline_P20.00x5.00mm_D1.05mm_Horizontal -> footprints:Fuseholder_Clip-5x20mm; Link https://jlcpcb.com/partdetail/XuchengElec-5x20/C3130 -> (none)
- L401: footprint Inductor_SMD:L_Sunlord_MWSA0503S -> footprints:SMD,10.4x10.3mm; Alternatywa https://jlcpcb.com/partdetail/10704-SMDRH105R2R2NT/C10164 -> (none); JLCPCB Part C920280 -> C10164; Link https://jlcpcb.com/partdetail/Coilcraft-XAL5030222MEC/C9202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 -> https://jlcpcb.com/partdetail/10704-SMDRH105R2R2NT/C10164; MFR Part XAL5030-222MEC -> SXN(Shun Xiang Nuo Elec); Manufacturer Coilcraft -> SMDRH105R-2R2NT
Other:
- note added: "https://webench.ti.com/power-designer/switching-regulator/customize/2?VinMin=4.5&VinMax=5.5&O1V=3.3&O1I=1&base_pn=LMR51430X&AppType=None&Flavor=None&op_TA=30&origin=pf_panel&lang_chosen=en-US&optfactor=3&Topology=Buck&flavor=None&VoltageOption=None"
- note added: "i2c addres 0x58"
- moved on the sheet: FID401, FID402, FID403, FID404, H401, H402, H403, H404

Commit message: pcb
Parts:
- added C410: 10u, Capacitor_SMD:C_1206_3216Metric, symbol Device:C
- J401: value J_SGP30 -> SGP30
- J402: value USB_C_Receptacle_USB2.0_16P -> USBC
- J404: value J_BMP1 -> BMP1
- J406: value J_BMP2 -> BMP2
- J408: value J_OLED -> OLED
- J409, J411: now not fitted
- TP401: footprint TestPoint:TestPoint_Pad_D1.5mm -> TestPoint:TestPoint_THTPad_D1.5mm_Drill0.7mm
- TP402: renamed from TP403; footprint TestPoint:TestPoint_Pad_D1.5mm -> TestPoint:TestPoint_THTPad_D1.5mm_Drill0.7mm
- TP403: renamed from TP402; footprint TestPoint:TestPoint_Pad_D1.5mm -> TestPoint:TestPoint_THTPad_D1.5mm_Drill0.7mm
Connections:
- net +3V3: now also J401.4 (Pin_4), J407.5 (Pin_5), C410.1; no longer J401.1 (Pin_1), J407.1 (Pin_1)
- net GND: now also J401.3 (Pin_3), J407.1 (Pin_1), C410.2; no longer J401.2 (Pin_2), J407.5 (Pin_5)
- net I2C_SCL: now also J401.2 (Pin_2); no longer J401.3 (Pin_3)
- net I2C_SDA: now also J401.1 (Pin_1); no longer J401.4 (Pin_4)
- net enc_S1_in: now also J407.2 (Pin_2); no longer J407.4 (Pin_4)
- net enc_key_in: now also J407.4 (Pin_4); no longer J407.2 (Pin_2)
Other:
- moved on the sheet: C404, J401, J407, TP403

Commit message: PCB routing
Parts:
- removed D401: D_Schottky_5A, Diode_SMD:D_SMA, symbol Device:D_Schottky
- J403: JLCPCB Part (none) -> C5155559; Link https://pl.aliexpress.com/item/33005175186.html?spm=a2g0o.p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 -> https://jlcpcb.com/partdetail/GSwitch-DC_005HD020/C5155559; MFR Part (none) -> DC-005H-D020; Manufacturer (none) -> G-Switch; now in the parts list
Connections:
- net at J403.1, TP401.1: now also F401.1
Other:
- moved on the sheet: TP401
Changed lines of the file:
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@@
 	)
 	(junction
-		(at 39.37 45.72)
+		(at 67.31 45.72)
 		(diameter 0)
 		(color 0 0 0 0)
 	)
 	(junction
-		(at 67.31 45.72)
+		(at 49.53 45.72)
 		(diameter 0)
 		(color 0 0 0 0)
@@
 	(wire
 		(pts
-			(xy 38.1 45.72) (xy 39.37 45.72)
+			(xy 38.1 45.72) (xy 49.53 45.72)
 		)
 		(stroke
@@
 	(wire
 		(pts
-			(xy 53.34 45.72) (xy 57.15 45.72)
-		)
-		(stroke
-			(width 0)
-			(type default)
-		)
-	)
-	(wire
-		(pts
 			(xy 199.39 34.29) (xy 198.12 34.29)
 		)
@@
 	(wire
 		(pts
-			(xy 39.37 45.72) (xy 45.72 45.72)
+			(xy 256.54 67.31) (xy 261.62 67.31)
 		)
 		(stroke
@@
 	(wire
 		(pts
-			(xy 256.54 67.31) (xy 261.62 67.31)
+			(xy 92.71 57.15) (xy 92.71 55.88)
 		)
 		(stroke
@@
 	(wire
 		(pts
-			(xy 92.71 57.15) (xy 92.71 55.88)
+			(xy 256.54 27.94) (xy 261.62 27.94)
 		)
 		(stroke
@@
 	(wire
 		(pts
-			(xy 256.54 27.94) (xy 261.62 27.94)
+			(xy 256.54 115.57) (xy 261.62 115.57)
 		)
 		(stroke
@@
 	(wire
 		(pts
-			(xy 256.54 115.57) (xy 261.62 115.57)
+			(xy 254 80.01) (xy 261.62 80.01)
 		)
 		(stroke
@@
 	(wire
 		(pts
-			(xy 254 80.01) (xy 261.62 80.01)
+			(xy 139.7 48.26) (xy 140.97 48.26)
 		)
 		(stroke
@@
 	(wire
 		(pts
-			(xy 139.7 48.26) (xy 140.97 48.26)
+			(xy 49.53 45.72) (xy 57.15 45.72)
 		)
 		(stroke
@@
 	(symbol
 		(lib_id "Connector:TestPoint")
-		(at 39.37 45.72 0)
+		(at 49.53 45.72 0)
 		(unit 1)
 		(exclude_from_sim no)
@@
 		(dnp no)
 		(property "Reference" "TP401"
-			(at 39.37 40.64 0)
+			(at 49.53 40.64 0)
 			(effects
 				(font
@@
 		)
 		(property "Value" "TestPoint"
-			(at 41.91 43.6879 0)
+			(at 52.07 43.6879 0)
 			(effects
 				(font
@@
 		)
 		(property "Footprint" "TestPoint:TestPoint_THTPad_D1.5mm_Drill0.7mm"
-			(at 44.45 45.72 0)
+			(at 54.61 45.72 0)
 			(effects
 				(font
@@
 		)
 		(property "Datasheet" "~"
-			(at 44.45 45.72 0)
+			(at 54.61 45.72 0)
 			(effects
 				(font
@@
 		)
 		(property "Description" "test point"
-			(at 39.37 45.72 0)
+			(at 49.53 45.72 0)
 			(effects
 				(font
@@
 		)
 		(property "Alternatywa" ""
-			(at 39.37 45.72 0)
+			(at 49.53 45.72 0)
 			(effects
 				(font
@@
 		)
 		(property "Sim.Type" ""
-			(at 39.37 45.72 0)
+			(at 49.53 45.72 0)
 			(effects
 				(font
@@
 	)
 	(symbol
-		(lib_id "Device:D_Schottky")
-		(at 49.53 45.72 180)
-		(unit 1)
-		(exclude_from_sim no)
-		(in_bom yes)
-		(on_board yes)
-		(dnp no)
-		(fields_autoplaced yes)
-		(property "Reference" "D401"
-			(at 49.8475 39.37 0)
-			(effects
-				(font
-					(size 1.27 1.27)
-				)
-			)
-		)
-		(property "Value" "D_Schottky_5A"
-			(at 49.8475 41.91 0)
-			(effects
-				(font
-					(size 1.27 1.27)
-				)
-			)
-		)
-		(property "Footprint" "Diode_SMD:D_SMA"
-			(at 49.53 45.72 0)
-			(effects
-				(font
-					(size 1.27 1.27)
-				)
-				(hide yes)
-			)
-		)
-		(property "Datasheet" "~"
-			(at 49.53 45.72 0)
-			(effects
-				(font
-					(size 1.27 1.27)
-				)
-				(hide yes)
-			)
-		)
-		(property "Description" "Schottky diode"
-			(at 49.53 45.72 0)
-			(effects
-				(font
-					(size 1.27 1.27)
-				)
-				(hide yes)
-			)
-		)
-		(property "Manufacturer" "MDD(Microdiode Semiconductor)"
-			(at 49.53 45.72 0)
-			(effects
-				(font
-					(size 1.27 1.27)
-				)
-				(hide yes)
-			)
-		)
-		(property "MFR Part" "SS34"
-			(at 49.53 45.72 0)
-			(effects
-				(font
-					(size 1.27 1.27)
-				)
-				(hide yes)
-			)
-		)
-		(property "Link" "https://jlcpcb.com/partdetail/MDD_Microdiode_Semiconductor-SS34/C8678"
-			(at 49.53 45.72 0)
-			(effects
-				(font
-					(size 1.27 1.27)
-				)
-				(hide yes)
-			)
-		)
-		(property "JLCPCB Part" "C8678"
-			(at 49.53 45.72 0)
-			(effects
-				(font
-					(size 1.27 1.27)
-				)
-				(hide yes)
-			)
-		)
-		(property "Alternatywa" ""
-			(at 49.53 45.72 0)
-			(effects
-				(font
-					(size 1.27 1.27)
-				)
-				(hide yes)
-			)
-		)
-		(property "Sim.Type" ""
-			(at 49.53 45.72 0)
-			(effects
-				(font
-					(size 1.27 1.27)
-				)
-				(hide yes)
-			)
-		)
-		(pin "2"
-		)
-		(pin "1"
-		)
-		(instances
-			(project "inz"
-				(path "/3ad3be82-7cab-4f72-ad1b-fa82ddc3a5e0/1dcd1198-aa22-4cf3-b3ba-8c43001473fa"
-					(reference "D401")
-					(unit 1)
-				)
-			)
-		)
-	)
-	(symbol
 		(lib_id "power:GND")
 		(at 242.57 160.02 0)
@@
 		(unit 1)
 		(exclude_from_sim no)
-		(in_bom no)
+		(in_bom yes)
 		(on_board yes)
 		(dnp no)
@@
 			)
 		)
-		(property "Link" "https://pl.aliexpress.com/item/33005175186.html?spm=a2g0o.productlist.main.2.46584999h0hQJo&algo_pvid=b1808c6d-ae88-44e2-b5d0-34e00a7523b1&algo_exp_id=b1808c6d-ae88-44e2-b5d0-34e00a7523b1-1&pdp_ext_f=%7B%22order%22%3A%22243%22%2C%22eval%22%3A%221%22%2C%22fromPage%22%3A%22search%22%7D&pdp_npi=6%40dis%21PLN%215.17%214.79%21%21%211.38%211.28%21%40211b61ae17645164079525576e2b82%2166974835404%21sea%21PL%212442407001%21X%211%210%21n_tag%3A-29919%3Bd%3A14685e7e%3Bm03_new_user%3A-29895&curPageLogUid=iN8p37Bcux95&utparam-url=scene%3Asearch%7Cquery_from%3A%7Cx_object_id%3A33005175186%7C_p_origin_prod%3A"
+		(property "Link" "https://jlcpcb.com/partdetail/GSwitch-DC_005HD020/C5155559"
 			(at 30.48 48.26 0)
 			(effects
@@
 			(at 30.48 48.26 0)
 			(effects
+				(font
+					(size 1.27 1.27)
+				)
+				(hide yes)
+			)
+		)
+		(property "JLCPCB Part" " C5155559"
+			(at 30.48 48.26 0)
+			(effects
+				(font
+					(size 1.27 1.27)
+				)
+				(hide yes)
+			)
+		)
+		(property "MFR Part" " DC-005H-D020"
+			(at 30.48 48.26 0)
+			(effects
+				(font
+					(size 1.27 1.27)
+				)
+				(hide yes)
+			)
+		)
+		(property "Manufacturer" " G-Switch"
+			(at 30.48 48.26 0)
+			(effects

Commit message: PCB final routing
Other:
- company: (none) -> Authors: D. Ledzianowski K. Lewandowska T. Majchrzak
Changed lines of the file:
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@@
 	(generator_version "9.0")
 	(paper "A4")
+	(title_block
+		(date "2025-12-07")
+		(rev "1.0")
+		(company "Authors: D. Ledzianowski K. Lewandowska T. Majchrzak")
+		(comment 2 "	")
+	)
 	(rectangle
 		(start 153.67 13.97)

Commit message: PCB final design
Parts:
- C402: JLCPCB Part C377773 -> C377773; MFR Part CL21A225KBQNNNE -> CL21A225KBQNNNE
- C403, C404: Manufacturer Samsung Electro-Mechanics -> Samsung Electro-Mechanics
- C409: Distributor https://jlcpcb.com/partdetail/29074-CL21B105KBFNNNE/C28323 -> (none)
- F401, J410: now not fitted
- J401: JLCPCB Part (none) -> C144395; Link https://pl.aliexpress.com/item/1005010374454394.html?spm=a2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 -> https://jlcpcb.com/partdetail/JST-B4B_XH_A_LF_SN/C144395; MFR Part (none) -> B4B-XH-A(LF)(SN); Manufacturer (none) -> JST
- J402: footprint Connector_USB:USB_C_Receptacle_GCT_USB4105-xx-A_16P_TopMnt_Horizontal -> footprints:USB_C_16P; JLCPCB Part C3025063 -> C47817612; Link https://jlcpcb.com/partdetail/3554049-USB4105_GF_A060/C3025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 -> https://jlcpcb.com/partdetail/Korean_HropartsElec-TYPE_C_31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; MFR Part USB4105-GF-A-060 -> TYPE-C-31-M-48; Manufacturer Global Connector Technology -> Korean Hroparts Elec
- J403: JLCPCB Part C5155559 -> C5155559; MFR Part DC-005H-D020 -> DC-005H-D020; Manufacturer G-Switch -> G-Switch
- J404: JLCPCB Part (none) -> C144397; Link https://pl.aliexpress.com/item/1005006960863510.html?spm=a2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 -> https://jlcpcb.com/partdetail/JST-B6B_XH_A_LF_SN/C144397; MFR Part (none) -> B6B-XH-A(LF)(SN); Manufacturer (none) -> JST; now in the parts list
- J405: Link https://pl.aliexpress.com/item/1005010319587802.html?spm=a2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 -> (none); now not fitted
- J406: JLCPCB Part (none) -> C144397; Link https://pl.aliexpress.com/item/1005006960863510.html?spm=a2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 -> https://jlcpcb.com/partdetail/JST-B6B_XH_A_LF_SN/C144397; MFR Part (none) -> B6B-XH-A(LF)(SN); Manufacturer (none) -> JST
- J407: JLCPCB Part (none) -> C157991; Link (none) -> https://jlcpcb.com/partdetail/JST-B5B_XH_A_LF_SN/C157991; MFR Part (none) -> B5B-XH-A(LF)(SN); Manufacturer (none) -> JST
- J408: JLCPCB Part (none) -> C157966; Link (none) -> https://jlcpcb.com/partdetail/JST-B9B_XH_A_LF_SN/C157966; MFR Part (none) -> B9B-XH-A(LF)(SN); Manufacturer (none) -> JST; now in the parts list
- J409: now in the parts list
- R401, R402, R404, R405, R406, R407: Manufacturer UNI-ROYAL(Uniroyal Elec) -> UNI-ROYAL(Uniroyal Elec)
- R403: Link https://jlcpcb.com/partdetail/28584-0805W8F5101T5E/C27834 -> https://jlcpcb.com/partdetail/160838-0805W8F1003T5E/C149504; MFR Part 0805W8F1003T5E -> 0805W8F1003T5E; Manufacturer UNI-ROYAL(Uniroyal Elec) -> UNI-ROYAL(Uniroyal Elec)
- R408, R409, R410, R411, R412: Distributor https://jlcpcb.com/partdetail/18102-0805W8F1002T5E/C17414 -> (none); JLCPCB Part C38522 -> C17414; Link https://jlcpcb.com/partdetail/39505-0805W8F1002T5E/C38522 -> https://jlcpcb.com/partdetail/18102-0805W8F1002T5E/C17414; MFR Part 0805W8F1002T5E -> 0805W8F1002T5E; Manufacturer UNI-ROYAL(Uniroyal Elec) -> UNI-ROYAL(Uniroyal Elec)
- U401: Manufacturer STMicroelectronics -> STMicroelectronics
