File: hardware/PCB/Connectors.kicad_sch (KiCad schematic)
At the start: 49 parts, among them J401 SGP30, J402 USBC, J403 5V, J404 BMP1, J406 BMP2, J407 enc, J408 OLED, J409 Conn_01x05_Pin, J410 Micro SD, J411 Micro SD2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

Commit message: usb, sd
Parts:
- F401, J405, J409, J410, J411: now fitted
Other:
- note added: "SMPS"
- note removed: "5.0V -> 3.3V"
- title: (none) -> Stanowisko do badania parametrów pracy ogniw Li-Ion Li-Pol
- moved on the sheet: C405, C406, C407, FID401, FID402, FID403, FID404, H401, H402, H403, H404, J407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
