File: hardware/PCB/inz.kicad_pcb (KiCad board)
At the start: 2 copper layers, 144 parts, among them J101 TP4056, J102 Battery, J103 STM32blackpill, J201 ina333, J202 ACS712, J301 BAT_LOAD, J302 J_BMP3, J303 100W 1R, J401 J_SGP30, J402 USB_C_Receptacle_USB2.0_16P, J403 5V, J404 J_BMP1, J406 J_BMP2, J407 enc, J408 J_OLED, J410 Micro SD, J411 Micro SD2, J412 Micro_SD_Card, J501 Screw_Terminal_01x03, J502 Screw_Terminal_01x03, J503 Screw_Terminal_01x03, J504 Relays_in, K501 SANYOU_SRD_Form_C, K502 SANYOU_SRD_Form_C, K503 SANYOU_SRD_Form_C, Q301 IRLZ44N, Q501 NPN, Q502 NPN, Q503 NPN, U201 INA333xxDGK, U202 MCP6002T-I/SN, U203 TLV431, U204 QNHC3, U205 TLV431, U206 ACS712xLCTR-05B, U301 LM358, U302 BME280, U401 USBLC6-2SC6, U402 LMR51430, U501 PC817C, U502 PC817C, U503 PC817C

Commit message: pcb
Parts:
- removed C302: 100n, Capacitor_SMD:C_0805_2012Metric
- removed C303: 10u, Capacitor_SMD:C_1206_3216Metric
- removed D503: 1N4148W, Diode_SMD:D_SOD-123
- removed J103: STM32blackpill, footprints:STM32blackpill
- removed J303: 100W 1R, TerminalBlock_Phoenix:TerminalBlock_Phoenix_MKDS-1,5-2_1x02_P5.00mm_Horizontal
- removed J502, J503: Screw_Terminal_01x03, TerminalBlock_Phoenix:TerminalBlock_Phoenix_MKDS-1,5-3_1x03_P5.00mm_Horizontal
- removed J504: Relays_in, Connector_PinHeader_2.54mm:PinHeader_1x06_P2.54mm_Vertical
- removed JP202: SolderJumper_3_Open, Jumper:SolderJumper-3_P2.0mm_Open_TrianglePad1.0x1.5mm_NumberLabels
- removed K501, K502, K503: SANYOU_SRD_Form_C, Relay_THT:Relay_SPDT_SANYOU_SRD_Series_Form_C
- removed Q503: NPN, Package_TO_SOT_SMD:SOT-23
- removed R505, R506: 220R, Resistor_SMD:R_0805_2012Metric
- removed U302: BME280, Package_LGA:Bosch_LGA-8_2.5x2.5mm_P0.65mm_ClockwisePinNumbering
- removed U503: PC817C, Package_DIP:DIP-4_W7.62mm_LongPads
- added C211: 100n, Capacitor_SMD:C_0805_2012Metric, F.Cu at (173.1, 95.0)
- added C212: 100n, Capacitor_SMD:C_0805_2012Metric, F.Cu at (175.1, 95.0)
- added C410: 10u, Capacitor_SMD:C_1206_3216Metric, F.Cu at (170.8, 48.7)
- added C601: 470u 50V, Capacitor_SMD:C_Elec_10x10.2, F.Cu at (61.1, 38.0)
- added C602: 1u, Capacitor_SMD:C_0805_2012Metric, F.Cu at (73.5, 29.0)
- added C603: 1u, Capacitor_SMD:C_0805_2012Metric, F.Cu at (77.0, 29.0)
- added C604: 1u, Capacitor_SMD:C_0805_2012Metric, F.Cu at (72.7, 49.5)
- added C605: 470u 50V, Capacitor_SMD:C_Elec_10x10.2, F.Cu at (86.0, 54.5)
- added C606: 1u, Capacitor_SMD:C_0805_2012Metric, F.Cu at (82.8, 68.8)
- added C607: 1u, Capacitor_SMD:C_0805_2012Metric, F.Cu at (65.0, 69.8)
- added C608: 10u, Capacitor_SMD:C_1206_3216Metric, F.Cu at (55.2, 64.0)
- added C609: 1u, Capacitor_SMD:C_0805_2012Metric, F.Cu at (63.4, 64.0)
- added C610: 1u, Capacitor_SMD:C_0805_2012Metric, F.Cu at (69.5, 64.0)
- added D601: MBRD1045, Diode_SMD:D_SMA, F.Cu at (69.6, 43.4)
- added D602: Red, LED_SMD:LED_0805_2012Metric, F.Cu at (85.5, 38.6)
- added D603: Yellow, LED_SMD:LED_0805_2012Metric, F.Cu at (56.1, 72.5)
- added D604: Green, LED_SMD:LED_0805_2012Metric, F.Cu at (60.1, 72.5)
- added J203: J_BMP3, Connector_JST:JST_XH_B6B-XH-A_1x06_P2.50mm_Vertical, F.Cu at (174.5, 88.5)
- added J409: Conn_01x05_Pin, Connector_JST:JST_XH_B5B-XH-A_1x05_P2.50mm_Vertical, F.Cu at (176.9, 103.6)
- added JP102: Jumper_2_Bridged, Connector_PinHeader_2.54mm:PinHeader_1x02_P2.54mm_Vertical, F.Cu at (75.0, 82.2)
- added JP201: SolderJumper_3_Open, Jumper:SolderJumper-3_P2.0mm_Open_TrianglePad1.0x1.5mm_NumberLabels, F.Cu at (78.5, 99.9)
- added K101: FRT5, Relay_THT:Relay_DPDT_FRT5, F.Cu at (108.8, 62.1)
- added K102: FRT5, Relay_THT:Relay_DPDT_FRT5, F.Cu at (108.8, 45.8)
- added L601: 47u, Inductor_THT:L_Toroid_Vertical_L16.0mm_W8.0mm_P7.62mm, F.Cu at (56.2, 53.0)
- added R601: 270, Resistor_SMD:R_0805_2012Metric, F.Cu at (85.5, 32.3)
- added R602: 1k, Resistor_SMD:R_0805_2012Metric, F.Cu at (56.1, 70.0)
- added R603: 2.2k, Resistor_SMD:R_0805_2012Metric, F.Cu at (67.3, 64.0)
- added R604: 71.5k, Resistor_SMD:R_0805_2012Metric, F.Cu at (77.0, 64.0)
- added R605: 90k9, Resistor_SMD:R_0805_2012Metric, F.Cu at (68.4, 74.8)
- added R606: 10k, Resistor_SMD:R_0805_2012Metric, F.Cu at (72.2, 74.8)
- added R607: 1k, Resistor_SMD:R_0805_2012Metric, F.Cu at (60.1, 70.0)
- added R608: 0.05R, Resistor_SMD:R_2512_6332Metric, F.Cu at (70.5, 78.0)
- added RV601: 10k, Potentiometer_THT:Potentiometer_Bourns_3299W_Vertical, F.Cu at (71.4, 56.4)
- added TP112: TestPoint, TestPoint:TestPoint_THTPad_D1.5mm_Drill0.7mm, F.Cu at (154.7, 80.9)
- added TP113: TestPoint, TestPoint:TestPoint_THTPad_D1.5mm_Drill0.7mm, F.Cu at (154.7, 83.7)
- added TP114: TestPoint, TestPoint:TestPoint_THTPad_D1.5mm_Drill0.7mm, F.Cu at (154.7, 86.4)
- added TP115: TestPoint, TestPoint:TestPoint_THTPad_D1.5mm_Drill0.7mm, F.Cu at (154.7, 89.2)
- added TP116: TestPoint, TestPoint:TestPoint_THTPad_D1.5mm_Drill0.7mm, F.Cu at (133.3, 90.0)
- added TP117: TestPoint, TestPoint:TestPoint_THTPad_D1.5mm_Drill0.7mm, F.Cu at (154.7, 91.9)
- added TP304: TestPoint, TestPoint:TestPoint_THTPad_D1.5mm_Drill0.7mm, F.Cu at (96.8, 29.1)
- added TP504: TestPoint, TestPoint:TestPoint_THTPad_D1.5mm_Drill0.7mm, F.Cu at (123.0, 56.4)
- added TP505: TestPoint, TestPoint:TestPoint_THTPad_D1.5mm_Drill0.7mm, F.Cu at (120.3, 56.4)
- added TP506: TestPoint, TestPoint:TestPoint_THTPad_D1.5mm_Drill0.7mm, F.Cu at (111.8, 57.6)
- added TP601: TestPoint, TestPoint:TestPoint_THTPad_D1.5mm_Drill0.7mm, F.Cu at (83.3, 27.4)
- added TP602: TestPoint, TestPoint:TestPoint_THTPad_D1.5mm_Drill0.7mm, F.Cu at (87.5, 67.0)
- added TP603: TestPoint, TestPoint:TestPoint_THTPad_D1.5mm_Drill0.7mm, F.Cu at (85.5, 35.2)
- added TP604: TestPoint, TestPoint:TestPoint_THTPad_D1.5mm_Drill0.7mm, F.Cu at (67.3, 60.2)
- added TP605: TestPoint, TestPoint:TestPoint_THTPad_D1.5mm_Drill0.7mm, F.Cu at (80.7, 62.3)
- added TP606: TestPoint, TestPoint:TestPoint_THTPad_D1.5mm_Drill0.7mm, F.Cu at (80.7, 65.0)
- added TP607: TestPoint, TestPoint:TestPoint_THTPad_D1.5mm_Drill0.7mm, F.Cu at (68.0, 29.0)
- added TP608: TestPoint, TestPoint:TestPoint_THTPad_D1.5mm_Drill0.7mm, F.Cu at (64.0, 73.0)
- added U207: BME280, Package_LGA:Bosch_LGA-8_2.5x2.5mm_P0.65mm_ClockwisePinNumbering, F.Cu at (169.3, 95.0)
- added U601: XL4015, Package_TO_SOT_SMD:TO-263-5_TabPin3, F.Cu at (77.5, 40.8)
- added U602: DS3502U+T&R, Package_SO:TSSOP-10_3x3mm_P0.5mm, F.Cu at (78.2, 68.8)
- added U603: LM358, Package_SO:SOIC-8_3.9x4.9mm_P1.27mm, F.Cu at (70.2, 71.0)
- added U604: 78L05, Package_TO_SOT_SMD:SOT-89-3, F.Cu at (59.2, 64.0)
- added U605: TL431, Package_TO_SOT_SMD:SOT-23-3, F.Cu at (73.8, 64.0)
- C301: value 100n -> 10u; footprint Capacitor_SMD:C_0805_2012Metric -> Capacitor_SMD:C_1206_3216Metric
- D401: value D_Schottky_3A -> D_Schottky_5A
- F401: value xA -> 5A; footprint Fuse:Fuseholder_Clip-5x20mm_Littelfuse_111_Inline_P20.00x5.00mm_D1.05mm_Horizontal -> footprints:Fuseholder_Clip-5x20mm
- J101: value TP4056 -> Battery; footprint footprints:board_TP4056 -> TerminalBlock_Phoenix:TerminalBlock_Phoenix_MKDS-1,5-2_1x02_P5.00mm_Horizontal
- J102: value Battery -> STM32blackpill; footprint TerminalBlock_Phoenix:TerminalBlock_Phoenix_MKDS-1,5-2_1x02_P5.00mm_Horizontal -> footprints:STM32blackpill
- J302: value J_BMP3 -> 100W 1R; footprint Connector_JST:JST_XH_B6B-XH-A_1x06_P2.50mm_Vertical -> TerminalBlock_Phoenix:TerminalBlock_Phoenix_MKDS-1,5-2_1x02_P5.00mm_Horizontal
- J401: value J_SGP30 -> SGP30
- J402: value USB_C_Receptacle_USB2.0_16P -> USB_C
- J404: value J_BMP1 -> BMP1
- J406: value J_BMP2 -> BMP2
- J408: value J_OLED -> OLED
- J501: value Screw_Terminal_01x03 -> Conn_01x04_Pin; footprint TerminalBlock_Phoenix:TerminalBlock_Phoenix_MKDS-1,5-3_1x03_P5.00mm_Horizontal -> Connector_PinHeader_2.54mm:PinHeader_1x04_P2.54mm_Vertical
- L401: footprint Inductor_SMD:L_Sunlord_MWSA0503S -> footprints:SMD,10.4x10.3mm
- TP101, TP102, TP103, TP104, TP105, TP106, TP107, TP108, TP109, TP110, TP111, TP201, TP202, TP203, TP204, TP205, TP206, TP207, TP301, TP302, TP303, TP401, TP402, TP403, TP501, TP502, TP503: footprint TestPoint:TestPoint_Pad_D1.5mm -> TestPoint:TestPoint_THTPad_D1.5mm_Drill0.7mm
- moved J406 129.0 mm to (174.8, 80.2), turned to 180 degrees
- moved J404 128.4 mm to (175.0, 72.0), turned to 180 degrees
- moved C301 116.5 mm to (92.3, 35.3), turned to 180 degrees
- moved J302 107.5 mm to (130.1, 31.0), turned to 180 degrees
- moved J102 96.7 mm to (136.4, 64.6), turned to 0 degrees
- moved TP104 77.0 mm to (110.2, 42.8), turned to 0 degrees
- moved TP101 70.6 mm to (108.8, 57.6), turned to -90 degrees
- moved TP102 69.3 mm to (106.2, 72.8), turned to 90 degrees
- moved TP103 67.7 mm to (106.2, 57.6), turned to 90 degrees
- moved J408 62.1 mm to (160.9, 103.6)
- moved J401 56.4 mm to (118.4, 103.6), turned to 180 degrees
- moved Q301 56.0 mm to (109.0, 28.2)
- moved J101 51.2 mm to (58.6, 80.0)
- moved J407 48.1 mm to (134.3, 103.6), turned to 180 degrees
- moved TP106 44.6 mm to (154.7, 51.4), turned to 0 degrees
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Connections:
- net /K2_NO renamed /BatteryLoad/Bat_load+
- net /Relays/K2_QC_K renamed /R2_COIL-
- C204 pad 1: /Current_sensor_in+ -> /Current_sensor_in-
- C301 pad 1: +3V3 -> /BatteryLoad/active_load_Vin+
- D501 pad 2: /Relays/K1_QC_K -> /R1_COIL-
- J101 pad 1: /K1_NO -> /BAT_Vin-
- J101 pad 2: GND -> /BAT_Vin+
- J102 pad 1: /ina333_Vin- -> /R1_IN1
- J102 pad 2: /Current_sensor_in+ -> /R1_IN2
- J201 pad 1: /Sensors1/ina333_Vref -> unconnected-(J201A-Vref-Pad1)
- J201 pad 8: /Current_sensor_in+ -> /Current_sensor_in-
- J302 pad 1: +3V3 -> GND
- J302 pad 2: GND -> /BatteryLoad/active_load_Vin-
- J401 pad 1: +3V3 -> /I2C_SDA
- J401 pad 2: GND -> /I2C_SCL
- J401 pad 3: /I2C_SCL -> GND
- J401 pad 4: /I2C_SDA -> +3V3
- J404 pad 4: /SPI_MISO -> /SPI_MOSI
- J404 pad 6: /SPI_MOSI -> /SPI_MISO
- J406 pad 4: /SPI_MISO -> /SPI_MOSI
- J406 pad 6: /SPI_MOSI -> /SPI_MISO
- J407 pad 1: +3V3 -> GND
- J407 pad 2: /Connectors/enc_key_in -> /Connectors/enc_S1_in
- J407 pad 4: /Connectors/enc_S1_in -> /Connectors/enc_key_in
- J407 pad 5: GND -> +3V3
- J408 pad 6: /SPI_MISO -> /SPI_MOSI
- J408 pad 8: /OLED_CS -> /OLED_TIM2
- J408 pad 9: /SPI_MOSI -> /SPI_MISO
- J410 pad 2: /SPI_MOSI -> /SPI_MISO
- J410 pad 4: /SPI_MISO -> /SPI_MOSI
- J411 pad 2: /SPI_MOSI -> /SPI_MISO
- J411 pad 4: /SPI_MISO -> /SPI_MOSI
- J412 pad 3: /SPI_MISO -> /SPI_MOSI
- J412 pad 7: /SPI_MOSI -> /SPI_MISO
- J501 pad 1: /K1_NC -> +5V
- J501 pad 2: +5V -> GND
- J501 pad 3: /K1_NO -> /R1_IN2
- JP101 pad 1: /Current_sensor_in+ -> /BAT_Vin+
- Q301 pad 1: /Sensors2/active_load_Vout -> /BatteryLoad/active_load_Vout
- Q301 pad 3: /Sensors2/active_load_Vin- -> /BatteryLoad/active_load_Vin-
- Q501 pad 1: /Relays/K1_QC_K -> /R1_COIL-
- R301 pad 2: /Sensors2/active_load_Vin+ -> /BatteryLoad/active_load_Vin+
- R410 pad 2: /SPI_MISO -> /SPI_MOSI
- R411 pad 2: /SPI_MOSI -> /SPI_MISO
- TP105 pad 1: Net-(J103B-PA0) -> /R1_IN3
- TP106 pad 1: Net-(J103B-RST) -> Net-(J102B-3V3)
- TP107 pad 1: Net-(J103B-PC15) -> Net-(J102A-PB15)
- TP108 pad 1: Net-(J103B-PC14) -> Net-(J102B-PB10)
- TP109 pad 1: Net-(J103B-PC13) -> Net-(J102B-PB2)
- TP110 pad 1: Net-(J103A-3V3) -> /TIM4_CH2
- TP111 pad 1: Net-(J103B-VB) -> Net-(J102B-PA0)
- TP301 pad 1: /Sensors2/active_load_Vin+ -> /TIM3_CH1_PWM
- TP302 pad 1: /Sensors2/active_load_Vout -> /BatteryLoad/active_load_Vin+
- TP303 pad 1: /Sensors2/active_load_Vin- -> /BatteryLoad/active_load_Vout
- TP402 pad 1: +3V3 -> +5V
- TP403 pad 1: +5V -> +3V3
- TP501 pad 1: /Relays/K1_opto_out -> +5V
- TP502 pad 1: /Relays/K2_opto_out -> /Relays/K1_opto_out
- TP503 pad 1: /Relays/K3_opto_out -> /R1_COIL-
- U201 pad 3: /Current_sensor_in+ -> /Current_sensor_in-
- U206 pad 1: /Current_sensor_in+ -> /Current_sensor_in-
- U206 pad 2: /Current_sensor_in+ -> /Current_sensor_in-
- U206 pad 3: /Current_sensor_in- -> /BAT_Vin+
- U206 pad 4: /Current_sensor_in- -> /BAT_Vin+
- U301 pad 1: /Sensors2/active_load_Vout -> /BatteryLoad/active_load_Vout
- U301 pad 2: /Sensors2/active_load_Vin- -> /BatteryLoad/active_load_Vin-
- U301 pad 3: /Sensors2/active_load_Vin+ -> /BatteryLoad/active_load_Vin+
Routing:
- net /Current_sensor_in-: track 0.00 -> 79.0 mm, vias 0 -> 8
- net /ina333_Vin-: track 0.00 -> 74.3 mm
- net GND: track 0.00 -> 42.7 mm
- net /BatteryLoad/active_load_Vin-: track 0.00 -> 36.9 mm, vias 0 -> 1
- net /BAT_Vin+: track 0.00 -> 22.2 mm
- net /BatteryLoad/active_load_Vout: track 0.00 -> 15.6 mm
- net /BAT_Vin-: track 0.00 -> 14.8 mm
- net /BatteryLoad/active_load_Vin+: track 0.00 -> 12.4 mm
- net /BatteryLoad/Bat_load+: track 0.00 -> 7.28 mm
- net Net-(K101-Pad2): track 0.00 -> 5.54 mm
- net Net-(K102-Pad9): track 0.00 -> 4.21 mm
- net /TIM3_CH1_PWM: track 0.00 -> 3.91 mm
- net Net-(K101-Pad9): track 0.00 -> 3.05 mm
- net /R1_COIL-: track 0.00 -> 3.00 mm
Other:
- board outline added: 140 x 85 mm
- board text added: "ACS712"
- board text added: "JLCJLCJLCJLC"

Commit message: pcb relay
Parts:
- J402: value USB_C -> USBC
- moved TP602 19.6 mm to (90.4, 47.6), turned to 0 degrees
- moved R608 19.5 mm to (86.3, 66.6), turned to -90 degrees
- moved TP205 14.0 mm to (72.8, 98.2)
- moved TP402 5.53 mm to (148.7, 27.3)
- moved TP601 5.27 mm to (88.3, 29.1), turned to 0 degrees
- moved TP607 4.08 mm to (64.0, 29.8), turned to 180 degrees
- moved TP203 3.77 mm to (122.5, 85.4)
- moved C602 3.74 mm to (70.4, 26.9), turned to 180 degrees
- moved TP605 2.81 mm to (80.7, 65.1)
- moved TP606 2.74 mm to (80.7, 62.3)
- moved TP207 2.58 mm to (122.5, 89.1)
- moved TP603 1.23 mm to (86.7, 35.4)
- moved D602 1.22 mm to (86.7, 38.5)
- moved R601 1.22 mm to (86.7, 32.3)
- moved C603 0.71 mm to (77.7, 29.1)
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Routing:
- net +5V: track 0.00 -> 201.6 mm, vias 0 -> 30
- net /XL4015/OUT+: track 0.00 -> 87.5 mm, vias 0 -> 8
- net /XL4015/OUT-: track 0.00 -> 63.8 mm, vias 0 -> 11
- net /XL4015/XL4015_ConstFlow_LED: track 0.00 -> 46.6 mm, vias 0 -> 2
- net /XL4015/XL4015_FB: track 0.00 -> 39.3 mm, vias 0 -> 1
- net /Sensors1/Current_sensor_out: track 0.00 -> 38.1 mm
- net /BatteryLoad/Bat_load+: track 7.28 -> 41.0 mm, vias 0 -> 9
- net /SPI_MISO: track 0.00 -> 30.8 mm
- net /XL4015/RVW: track 0.00 -> 28.5 mm
- net /R1_IN2: track 0.00 -> 28.4 mm
- net /XL4015/XL4015_5V: track 0.00 -> 27.2 mm
- net /R1_IN1: track 0.00 -> 26.4 mm
- net +3V3: track 0.00 -> 26.3 mm
- net /Sensors1/ACS712_out: track 0.00 -> 26.2 mm
- net /XL4015/XL4015_SW: track 0.00 -> 25.7 mm
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- added copper zone on F.Cu, net +5V
- added copper zone on F.Cu, net /XL4015/XL4015_SW
- added copper zone on B.Cu, net GND
- added copper zone on F.Cu, net GND
Other:
- outline, holes or cut-outs redrawn

Commit message: PCB routing
Parts:
- removed D401: D_Schottky_5A, Diode_SMD:D_SMA
- removed K101, K102: FRT5, Relay_THT:Relay_DPDT_FRT5
- added RL101: JW2, Relay_THT:Relay_DPDT_Panasonic_JW2, F.Cu at (121.8, 61.0)
- added RL102: JW2, Relay_THT:Relay_DPDT_Panasonic_JW2, F.Cu at (121.8, 43.8)
- moved J501 13.7 mm to (133.4, 39.2), turned to 90 degrees
- moved TP503 13.0 mm to (121.8, 72.8)
- moved TP402 12.4 mm to (136.3, 27.6)
- moved D501 11.8 mm to (126.5, 62.2)
- moved D502 11.8 mm to (126.8, 44.9)
- moved Q501 11.8 mm to (127.4, 68.3)
- moved Q502 11.8 mm to (127.7, 50.8)
- moved R502 11.8 mm to (127.4, 72.1)
- moved R504 11.8 mm to (127.7, 54.6)
- moved U501 11.0 mm to (134.1, 62.2)
- moved R503 11.0 mm to (133.3, 43.3)
- moved TP504 11.0 mm to (134.0, 56.6)
- moved TP505 11.0 mm to (131.3, 56.6)
- moved U502 11.0 mm to (134.0, 45.9)
- moved R501 11.0 mm to (133.2, 59.5)
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Connections:
- F401 pad 1: Net-(D401-K) -> Net-(F401-Pad1)
- J403 pad 1: Net-(D401-A) -> Net-(F401-Pad1)
- TP401 pad 1: Net-(D401-A) -> Net-(F401-Pad1)
Routing:
- net +3V3: track 26.3 -> 424.5 mm, vias 0 -> 13
- net +5V: track 201.6 -> 531.8 mm, vias 30 -> 34
- net /I2C_SDA: track 0.00 -> 134.6 mm, vias 0 -> 1
- net /I2C_SCL: track 0.00 -> 134.3 mm, vias 0 -> 1
- net /SPI_MOSI: track 23.1 -> 139.9 mm, vias 0 -> 2
- net /SPI_MISO: track 30.8 -> 146.2 mm
- net GND: track 54.2 -> 163.0 mm, vias 24 -> 82
- net /TIM3_CH1_PWM: track 4.04 -> 110.2 mm, vias 0 -> 2
- net /SPI_SCK: track 22.3 -> 119.8 mm, vias 0 -> 2
- net /SD_CS: track 0.00 -> 71.2 mm, vias 0 -> 2
- net /enc_KEY: track 2.02 -> 59.2 mm, vias 0 -> 1
- net /enc_S2: track 2.02 -> 58.6 mm, vias 0 -> 1
- net /enc_S1: track 2.02 -> 57.7 mm, vias 0 -> 1
- net /QNH_Vout: track 10.7 -> 58.2 mm, vias 0 -> 1
- net USB_D+: track 0.00 -> 47.1 mm, vias 0 -> 1
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- added copper zone on F.Cu, net +3V3
- added copper zone on B.Cu, net +5V
- added copper zone on F.Cu, net /Connectors/SMPS_SW
- added copper zone on B.Cu, net Net-(F401-Pad1)
- added copper zone on F.Cu, net Net-(F401-Pad1)

Commit message: PCB final routing
Parts:
- moved TP402 1.90 mm to (134.4, 27.5)
Routing:
- net GND: track 163.0 -> 177.1 mm, vias 82 -> 302
- net +5V: track 531.8 -> 540.6 mm
- net /SPI_MISO: track 146.2 -> 147.6 mm
- net +3V3: track 424.5 -> 425.5 mm
Other:
- board text added: "Authors: D. Ledzianowski K. Lewandowska T. Majchrzak"
- board text added: "Rev: 1.0"

Commit message: PCB final design
Parts:
- removed C211, C212: 100n, Capacitor_SMD:C_0805_2012Metric
- removed U207: BME280, Package_LGA:Bosch_LGA-8_2.5x2.5mm_P0.65mm_ClockwisePinNumbering
- C601, C605: value 470u 50V -> 470u
- J102: footprint footprints:STM32blackpill -> Package_DIP:DIP-40_W15.24mm
- J203: value J_BMP3 -> BMP3; footprint Connector_JST:JST_XH_B6B-XH-A_1x06_P2.50mm_Vertical -> Connector_PinHeader_2.54mm:PinHeader_1x06_P2.54mm_Vertical
- J302: value 100W 1R -> 1R 100W
- J402: footprint Connector_USB:USB_C_Receptacle_GCT_USB4105-xx-A_16P_TopMnt_Horizontal -> footprints:USB_C_16P
- R605: value 90k9 -> 90.9k
- U501, U502: value PC817C -> LTV-217; footprint Package_DIP:DIP-4_W7.62mm_LongPads -> Package_SO:SOP-4_4.4x2.6mm_P1.27mm
- moved J102 22.9 mm to (141.2, 45.9)
- moved U501 4.06 mm to (132.5, 66.0)
- moved U502 3.42 mm to (132.5, 49.0)
- moved J403 2.73 mm to (183.0, 38.9)
- moved R502 2.14 mm to (127.9, 70.0)
- moved Q501 1.92 mm to (127.9, 66.5)
- moved R504 1.62 mm to (127.9, 53.0)
- moved TP504 1.54 mm to (133.8, 55.0)
- moved TP505 1.54 mm to (131.1, 55.0)
- moved D501 1.49 mm to (127.0, 60.9)
- moved TP401 1.45 mm to (178.2, 45.5)
- moved Q502 1.34 mm to (127.9, 49.5)
- moved TP501 1.10 mm to (133.8, 72.0)
- moved TP502 1.10 mm to (131.1, 72.0)
- moved D502 1.09 mm to (127.0, 43.9)
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Connections:
- J102 pad 21: +5V -> Net-(J102B-VB)
- J102 pad 22: GND -> Net-(J102B-PC13)
- J102 pad 23: Net-(J102B-3V3) -> Net-(J102B-PC14)
- J102 pad 24: Net-(J102B-PB10) -> Net-(J102B-PC15)
- J102 pad 25: Net-(J102B-PB2) -> Net-(J102B-RST)
- J102 pad 26: /ina333_Vout -> Net-(J102B-PA0)
- J102 pad 27: /QNH_Vout -> /OLED_CS
- J102 pad 28: /SPI_MOSI -> /OLED_DC
- J102 pad 29: /SPI_MISO -> /OLED_RST
- J102 pad 30: /SPI_SCK -> /SD_CS
- J102 pad 31: /SD_CS -> /SPI_SCK
- J102 pad 32: /OLED_RST -> /SPI_MISO
- J102 pad 33: /OLED_DC -> /SPI_MOSI
- J102 pad 34: /OLED_CS -> /QNH_Vout
- J102 pad 35: Net-(J102B-PA0) -> /ina333_Vout
- J102 pad 36: Net-(J102B-RST) -> Net-(J102B-PB2)
- J102 pad 37: Net-(J102B-PC15) -> Net-(J102B-PB10)
- J102 pad 38: Net-(J102B-PC14) -> Net-(J102B-3V3)
- J102 pad 39: Net-(J102B-PC13) -> GND
- J102 pad 40: Net-(J102B-VB) -> +5V
Routing:
- net /SPI_MISO: track 147.6 -> 132.0 mm
- net +3V3: track 425.5 -> 410.8 mm
- net Net-(F401-Pad1): track 23.6 -> 13.5 mm, vias 11 -> 2
- net /BMP3_CS: track 36.6 -> 28.5 mm
- net /SPI_MOSI: track 139.9 -> 133.2 mm
- net /SPI_SCK: track 119.8 -> 114.1 mm
- net +5V: track 540.6 -> 537.3 mm
- net GND: track 177.1 -> 174.6 mm, vias 302 -> 319
- net /R1_IN1: track 25.0 -> 26.6 mm
- net /Relays/K1_opto_out: track 7.45 -> 5.93 mm
- net /SD_CS: track 71.2 -> 69.9 mm
- net /R1_COIL-: track 13.0 -> 14.3 mm
- net /R1_IN2: track 18.1 -> 19.4 mm
- net /Sensors1/ina333_Rg2: track 4.81 -> 3.59 mm
- net /R2_COIL-: track 13.1 -> 14.2 mm
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- removed copper zone on B.Cu, net Net-(F401-Pad1)

Commit message: oled, sd
Parts:
- J102: footprint Package_DIP:DIP-40_W15.24mm -> footprints:STM32blackpill
- moved J102 22.9 mm to (141.2, 68.8)
