File: hardware/PCB/BatteryLoad.kicad_sch (KiCad schematic)
At the start: 11 parts, among them J301 BAT_LOAD, J303 100W 1R, Q301 IRLZ44N, U301 LM358

Commit message: pcb
Parts:
- removed H405, H406: ResistorMountingHole, MountingHole:MountingHole_3.2mm_M3_Pad, symbol Mechanical:MountingHole
- added TP301: TestPoint, TestPoint:TestPoint_THTPad_D1.5mm_Drill0.7mm, symbol Connector:TestPoint
- J301: now not fitted
- TP302: renamed from TP301; footprint TestPoint:TestPoint_Pad_D1.5mm -> TestPoint:TestPoint_THTPad_D1.5mm_Drill0.7mm
- TP303: renamed from TP302; footprint TestPoint:TestPoint_Pad_D1.5mm -> TestPoint:TestPoint_THTPad_D1.5mm_Drill0.7mm
- TP304: renamed from TP303; footprint TestPoint:TestPoint_Pad_D1.5mm -> TestPoint:TestPoint_THTPad_D1.5mm_Drill0.7mm
- renumbered C303 to C301, J303 to J302
Connections:
- net GND: now also J302.1 (Pin_1); no longer J302.2 (Pin_2)
- net active_load_Vin-: now also J302.2 (Pin_2); no longer J302.1 (Pin_1)
- net pwm_current_sel: now also TP301.1

Commit message: PCB final routing
Other:
- company: (none) -> Authors: D. Ledzianowski K. Lewandowska T. Majchrzak
Changed lines of the file:
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@@
 	(generator_version "9.0")
 	(paper "A4")
+	(title_block
+		(date "2025-12-07")
+		(rev "1.0")
+		(company "Authors: D. Ledzianowski K. Lewandowska T. Majchrzak")
+	)
 	(text "Uniwersalne obciazenie aktywne"
 		(exclude_from_sim no)

Commit message: PCB final design
Parts:
- J302: value 100W 1R -> 1R 100W; now not fitted
- Q301: JLCPCB Part C38774 -> C38774; MFR Part IRLZ44NPBF -> IRLZ44NPBF; Manufacturer Infineon Technologies -> Infineon Technologies
Changed lines of the file:
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@@
 			)
 		)
-		(property "JLCPCB Part" " C38774"
+		(property "JLCPCB Part" "C38774"
 			(at 160.02 92.71 0)
 			(effects
@@
 			)
 		)
-		(property "MFR Part" " IRLZ44NPBF"
+		(property "MFR Part" "IRLZ44NPBF"
 			(at 160.02 92.71 0)
 			(effects
@@
 			)
 		)
-		(property "Manufacturer" " Infineon Technologies"
+		(property "Manufacturer" "Infineon Technologies"
 			(at 160.02 92.71 0)
 			(effects
@@
 		(in_bom no)
 		(on_board yes)
-		(dnp no)
+		(dnp yes)
 		(property "Reference" "J302"
 			(at 170.688 113.284 0)
@@
 			)
 		)
-		(property "Value" "100W 1R"
+		(property "Value" "1R 100W"
 			(at 170.688 110.744 0)
 			(effects

Commit message: oled, sd
Parts:
- J301, J302: now fitted
Other:
- moved on the sheet: C301, Q301, R301, TP302, TP303, TP304, U301A

Commit message: usb, sd
Other:
- title: (none) -> Stanowisko do badania parametrów pracy ogniw Li-Ion Li-Pol
- moved on the sheet: J301
Changed lines of the file:
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@@
 	(paper "A4")
 	(title_block
-		(date "2025-12-07")
-		(rev "1.0")
+		(title "Stanowisko do badania parametrów pracy ogniw Li-Ion Li-Pol")
+		(date "2025-12-10")
+		(rev "0.1")
 		(company "Authors: D. Ledzianowski K. Lewandowska T. Majchrzak")
 	)
@@
 	(text "Bat-"
 		(exclude_from_sim no)
-		(at 200.152 100.838 0)
+		(at 173.482 100.838 0)
 		(effects
 			(font
@@
 	(text "Bat+"
 		(exclude_from_sim no)
-		(at 200.152 92.456 0)
+		(at 173.482 92.456 0)
 		(effects
 			(font
@@
 	)
 	(junction
-		(at 195.58 88.9)
+		(at 168.91 88.9)
 		(diameter 0)
 		(color 0 0 0 0)
@@
 	)
 	(junction
-		(at 195.58 104.14)
+		(at 168.91 104.14)
 		(diameter 0)
 		(color 0 0 0 0)
@@
 	(wire
 		(pts
-			(xy 195.58 88.9) (xy 195.58 80.01)
+			(xy 168.91 88.9) (xy 168.91 80.01)
 		)
 		(stroke
@@
 	(wire
 		(pts
-			(xy 195.58 88.9) (xy 196.85 88.9)
-		)
-		(stroke
-			(width 0)
-			(type default)
-		)
-	)
-	(wire
-		(pts
-			(xy 195.58 104.14) (xy 196.85 104.14)
+			(xy 148.59 80.01) (xy 148.59 87.63)
+		)
+		(stroke
+			(width 0)
+			(type default)
+		)
+	)
+	(wire
+		(pts
+			(xy 168.91 88.9) (xy 170.18 88.9)
+		)
+		(stroke
+			(width 0)
+			(type default)
+		)
+	)
+	(wire
+		(pts
+			(xy 168.91 104.14) (xy 170.18 104.14)
 		)
 		(stroke
@@
 	(wire
 		(pts
-			(xy 195.58 95.25) (xy 195.58 88.9)
+			(xy 168.91 95.25) (xy 168.91 88.9)
 		)
 		(stroke
@@
 	(wire
 		(pts
-			(xy 195.58 104.14) (xy 195.58 113.03)
+			(xy 168.91 104.14) (xy 168.91 113.03)
 		)
 		(stroke
@@
 	(wire
 		(pts
-			(xy 148.59 113.03) (xy 195.58 113.03)
-		)
-		(stroke
-			(width 0)
-			(type default)
-		)
-	)
-	(wire
-		(pts
 			(xy 119.38 114.3) (xy 119.38 113.03)
 		)
@@
 	(wire
 		(pts
-			(xy 195.58 97.79) (xy 195.58 104.14)
+			(xy 168.91 97.79) (xy 168.91 104.14)
 		)
 		(stroke
@@
 	(wire
 		(pts
-			(xy 148.59 80.01) (xy 195.58 80.01)
+			(xy 148.59 80.01) (xy 168.91 80.01)
 		)
 		(stroke
@@
 	(wire
 		(pts
-			(xy 148.59 80.01) (xy 148.59 87.63)
-		)
-		(stroke
-			(width 0)
-			(type default)
-		)
-	)
-	(wire
-		(pts
 			(xy 132.08 92.71) (xy 140.97 92.71)
 		)
@@
 		)
 	)
+	(wire
+		(pts
+			(xy 148.59 113.03) (xy 168.91 113.03)
+		)
+		(stroke
+			(width 0)
+			(type default)
+		)
+	)
 	(label "Bat_load+"
-		(at 149.86 80.01 0)
+		(at 166.37 80.01 0)
 		(effects
 			(font
@@
 	(hierarchical_label "Bat_load+"
 		(shape input)
-		(at 196.85 88.9 0)
+		(at 170.18 88.9 0)
 		(effects
 			(font
@@
 	(hierarchical_label "Bat_load-"
 		(shape input)
-		(at 196.85 104.14 0)
+		(at 170.18 104.14 0)
 		(effects
 			(font
@@
 	(symbol
 		(lib_id "Connector_Generic:Conn_01x02")
-		(at 200.66 95.25 0)
+		(at 173.99 95.25 0)
 		(unit 1)
 		(exclude_from_sim no)
@@
 		(fields_autoplaced yes)
 		(property "Reference" "J301"
-			(at 203.2 95.2499 0)
+			(at 176.53 95.2499 0)
 			(effects
 				(font
@@
 		)
 		(property "Value" "BAT_LOAD"
-			(at 203.2 97.7899 0)
+			(at 176.53 97.7899 0)
 			(effects
 				(font
@@
 		)
 		(property "Footprint" "TerminalBlock:TerminalBlock_MaiXu_MX126-5.0-02P_1x02_P5.00mm"
-			(at 200.66 95.25 0)
+			(at 173.99 95.25 0)
 			(effects
 				(font
@@
 		)
 		(property "Datasheet" "~"
-			(at 200.66 95.25 0)
+			(at 173.99 95.25 0)
 			(effects
 				(font
@@
 		)
 		(property "Description" "Generic connector, single row, 01x02, script generated (kicad-library-utils/schlib/autogen/connector/)"
-			(at 200.66 95.25 0)
+			(at 173.99 95.25 0)
 			(effects
 				(font
@@
 		)
 		(property "Alternatywa" ""
-			(at 200.66 95.25 0)
+			(at 173.99 95.25 0)
 			(effects
 				(font
@@
 		)
 		(property "Sim.Type" ""
-			(at 200.66 95.25 0)
-			(effects
-				(font
+			(at 173.99 95.25 0)
+			(effects
+				(font
