File: hardware/PCB/XL4015.kicad_sch (KiCad schematic)
At the start: 36 parts, among them U1 XL4015, U2 78L05, U3 TL431, U303 DS3502U+T&R, U4 LM358

Commit message: pcb
Parts:
- removed TP306: TestPoint, TestPoint:TestPoint_Pad_D1.5mm, symbol Connector:TestPoint
- added TP601, TP607: TestPoint, TestPoint:TestPoint_THTPad_D1.5mm_Drill0.7mm, symbol Connector:TestPoint
- TP602: renamed from TP304; footprint TestPoint:TestPoint_Pad_D1.5mm -> TestPoint:TestPoint_THTPad_D1.5mm_Drill0.7mm
- TP603: renamed from TP307; footprint TestPoint:TestPoint_Pad_D1.5mm -> TestPoint:TestPoint_THTPad_D1.5mm_Drill0.7mm
- TP604: renamed from TP308; footprint TestPoint:TestPoint_Pad_D1.5mm -> TestPoint:TestPoint_THTPad_D1.5mm_Drill0.7mm
- TP605: renamed from TP310; footprint TestPoint:TestPoint_Pad_D1.5mm -> TestPoint:TestPoint_THTPad_D1.5mm_Drill0.7mm
- TP606: renamed from TP309; footprint TestPoint:TestPoint_Pad_D1.5mm -> TestPoint:TestPoint_THTPad_D1.5mm_Drill0.7mm
- TP608: renamed from TP305; footprint TestPoint:TestPoint_Pad_D1.5mm -> TestPoint:TestPoint_THTPad_D1.5mm_Drill0.7mm
- renumbered C1 to C601, C2 to C602, C3 to C603, C4 to C604, C5 to C605, C304 to C606, C9 to C607, C6 to C608, C7 to C609, C8 to C610, D1 to D601, D2 to D602, D4 to D603, D3 to D604, L1 to L601, R2 to R601, R1 to R602, R3 to R603, R4 to R604, R7 to R605, R6 to R606, R5 to R607, R9 to R608, RV301 to RV601, U1 to U601, U303 to U602, U4 to U603, U2 to U604, U3 to U605
Connections:
- net IN+: now also TP601.1
- net IN-: now also TP607.1
Other:
- moved on the sheet: TP602

Commit message: PCB final routing
Other:
- company: (none) -> Authors: D. Ledzianowski K. Lewandowska T. Majchrzak
Changed lines of the file:
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@@
 	(generator_version "9.0")
 	(paper "A4")
+	(title_block
+		(date "2025-12-07")
+		(rev "1.0")
+		(company "Authors: D. Ledzianowski K. Lewandowska T. Majchrzak")
+	)
 	(text "i2c addres 0x28"
 		(exclude_from_sim no)

Commit message: PCB final design
Parts:
- C601, C605: value 470u 50V -> 470u; JLCPCB Part C2887271 -> C3351; Link https://jlcpcb.com/partdetail/KNSCHA-RVT220UF50V67RV0021/C2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 -> https://jlcpcb.com/partdetail/HonorElec-RVT1E471M1010/C3351; MFR Part RVT220UF50V67RV0021 -> RVT1E471M1010; Manufacturer KNSCHA -> Honor Elec
- D602: JLCPCB Part C84256 -> C84256; MFR Part NCD0805R1 -> NCD0805R1
- D603: JLCPCB Part C2296 -> C2296; MFR Part KT-0805Y -> KT-0805Y; Manufacturer Hubei KENTO Elec -> Hubei KENTO Elec
- D604: JLCPCB Part C2297 -> C2297; MFR Part KT-0805G -> KT-0805G; Manufacturer Hubei KENTO Elec -> Hubei KENTO Elec
- R601: JLCPCB Part (none) -> C17590; Link (none) -> https://jlcpcb.com/partdetail/18278-0805W8F2700T5E/C17590; MFR Part (none) -> 0805W8F2700T5E; Manufacturer (none) -> UNI-ROYAL(Uniroyal Elec)
- R605: value 90k9 -> 90.9k
- R606: JLCPCB Part C38522 -> C17414; MFR Part 0805W8F1002T5E -> 0805W8F1002T5E; Manufacturer UNI-ROYAL(Uniroyal Elec) -> UNI-ROYAL(Uniroyal Elec)
- R608: Manufacturer UNI-ROYAL(Uniroyal Elec) -> UNI-ROYAL(Uniroyal Elec)
- RV601: now not fitted
- U601: JLCPCB Part C51661 -> C51661; Manufacturer XLSEMI -> XLSEMI
Changed lines of the file:
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@@
 		(in_bom no)
 		(on_board yes)
-		(dnp no)
+		(dnp yes)
 		(fields_autoplaced yes)
 		(property "Reference" "RV601"
@@
 			)
 		)
-		(property "JLCPCB Part" " C2297"
+		(property "JLCPCB Part" "C2297"
 			(at 166.37 115.57 90)
 			(effects
@@
 			)
 		)
-		(property "MFR Part" " KT-0805G"
+		(property "MFR Part" "KT-0805G"
 			(at 166.37 115.57 90)
 			(effects
@@
 			)
 		)
-		(property "Manufacturer" " Hubei KENTO Elec"
+		(property "Manufacturer" "Hubei KENTO Elec"
 			(at 166.37 115.57 90)
 			(effects
@@
 			)
 		)
-		(property "JLCPCB Part" " C51661"
+		(property "JLCPCB Part" "C51661"
 			(at 102.87 72.39 0)
 			(effects
@@
 			)
 		)
-		(property "Manufacturer" " XLSEMI"
+		(property "Manufacturer" "XLSEMI"
 			(at 102.87 72.39 0)
 			(effects
@@
 			)
 		)
-		(property "JLCPCB Part" " C2296"
+		(property "JLCPCB Part" "C2296"
 			(at 157.48 102.87 90)
 			(effects
@@
 			)
 		)
-		(property "MFR Part" " KT-0805Y"
+		(property "MFR Part" "KT-0805Y"
 			(at 157.48 102.87 90)
 			(effects
@@
 			)
 		)
-		(property "Manufacturer" " Hubei KENTO Elec"
+		(property "Manufacturer" "Hubei KENTO Elec"
 			(at 157.48 102.87 90)
 			(effects
@@
 			)
 		)
-		(property "Value" "470u 50V"
+		(property "Value" "470u"
 			(at 60.96 75.3109 0)
 			(effects
@@
 			)
 		)
-		(property "JLCPCB Part" "C2887271"
+		(property "JLCPCB Part" "C3351"
 			(at 64.77 74.93 0)
 			(effects
@@
 			)
 		)
-		(property "Link" "https://jlcpcb.com/partdetail/KNSCHA-RVT220UF50V67RV0021/C2887271"
+		(property "Link" "https://jlcpcb.com/partdetail/HonorElec-RVT1E471M1010/C3351"
 			(at 64.77 74.93 0)
 			(effects
@@
 			)
 		)
-		(property "MFR Part" "RVT220UF50V67RV0021"
+		(property "MFR Part" "RVT1E471M1010"
 			(at 64.77 74.93 0)
 			(effects
@@
 			)
 		)
-		(property "Manufacturer" " KNSCHA"
+		(property "Manufacturer" "Honor Elec"
 			(at 64.77 74.93 0)
 			(effects
@@
 			)
 		)
-		(property "Manufacturer" " UNI-ROYAL(Uniroyal Elec)"
+		(property "Manufacturer" "UNI-ROYAL(Uniroyal Elec)"
 			(at 151.13 137.16 90)
 			(effects
@@
 			)
 		)
-		(property "Value" "90k9"
+		(property "Value" "90.9k"
 			(at 139.7 124.714 90)
 			(effects
@@
 			)
 		)
-		(property "Value" "470u 50V"
+		(property "Value" "470u"
 			(at 158.75 75.3109 0)
 			(effects
@@
 			)
 		)
-		(property "JLCPCB Part" "C2887271"
+		(property "JLCPCB Part" "C3351"
 			(at 154.94 74.93 0)
 			(effects
@@
 			)
 		)
-		(property "Link" "https://jlcpcb.com/partdetail/KNSCHA-RVT220UF50V67RV0021/C2887271"
+		(property "Link" "https://jlcpcb.com/partdetail/HonorElec-RVT1E471M1010/C3351"
 			(at 154.94 74.93 0)
 			(effects
@@
 			)
 		)
-		(property "MFR Part" "RVT220UF50V67RV0021"
+		(property "MFR Part" "RVT1E471M1010"
 			(at 154.94 74.93 0)
 			(effects
@@
 			)
 		)
-		(property "Manufacturer" " KNSCHA"
+		(property "Manufacturer" "Honor Elec"
 			(at 154.94 74.93 0)
 			(effects
@@
 			)
 		)
-		(property "JLCPCB Part" " C84256"
+		(property "JLCPCB Part" "C84256"
 			(at 124.46 95.25 0)
 			(effects
@@
 			)
 		)
-		(property "MFR Part" " NCD0805R1"
+		(property "MFR Part" "NCD0805R1"
 			(at 124.46 95.25 0)
 			(effects
@@
 			)
 		)
-		(property "MFR Part" "0805W8F1002T5E "
+		(property "MFR Part" "0805W8F1002T5E"
 			(at 139.7 130.81 0)
 			(effects
@@
 			)
 		)
-		(property "Manufacturer" "UNI-ROYAL(Uniroyal Elec) "
+		(property "Manufacturer" "UNI-ROYAL(Uniroyal Elec)"
 			(at 139.7 130.81 0)
 			(effects
@@
 			)
 		)
-		(property "JLCPCB Part" "C38522"
+		(property "JLCPCB Part" "C17414"
 			(at 139.7 130.81 0)
 			(effects
@@
 			)
 		)
-		(property "MFR Part" ""
+		(property "MFR Part" "0805W8F2700T5E"
 			(at 132.08 93.98 0)
 			(effects
@@
 			)
 		)
-		(property "Manufacturer" ""
+		(property "Manufacturer" "UNI-ROYAL(Uniroyal Elec)"
 			(at 132.08 93.98 0)
 			(effects
@@
 			)
 		)
-		(property "JLCPCB Part" ""
+		(property "JLCPCB Part" "C17590"
 			(at 132.08 93.98 0)
 			(effects
@@
 			(at 132.08 93.98 0)
 			(effects
+				(font
+					(size 1.27 1.27)
+				)
+				(hide yes)
+			)
+		)
+		(property "Link" "https://jlcpcb.com/partdetail/18278-0805W8F2700T5E/C17590"
+			(at 132.08 93.98 0)
+			(effects

Commit message: usb, sd
Parts:
- RV601: now fitted
Other:
- title: (none) -> Stanowisko do badania parametrów pracy ogniw Li-Ion Li-Pol
- moved on the sheet: C601, C602, C603, C604, C605, C606, C607, C608, C609, C610, D601, D602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
